File: pcb/openxcvr/RADIO.kicad_pcb (KiCad board)
At the start: 2 copper layers, 99.1 x 63.5 mm, 121 parts, among them J1 UI_CONNECTOR, J2 PA_CONNECTOR, J3 GPS_CONNECTOR, J4 TEST_SIGNAL_CONNECTOR, U1 SN74CBT3253, U10 SN74CBT3253, U11 24LC256, U2 LM4562, U3 LM4562, U4 LM4562, U5 LM386, U6 MCP6002-xSN, U7 PCM1802, U8 MAX_1000, U9 SN74CBT3253

Commit message: Candidate design
Parts:
- removed the C1 at (122.6, 75.6)
- removed the C23 at (144.8, 94.3)
- removed the C24 at (132.1, 94.3)
- removed J4: TEST_SIGNAL_CONNECTOR, Connector_PinHeader_2.54mm:PinHeader_1x02_P2.54mm_Vertical
- removed the R2 at (122.6, 73.0)
- removed the U2 at (138.4, 61.0)
- removed the U4 at (138.3, 77.5)
- added C53: 100n, Capacitor_SMD:C_0805_2012Metric, F.Cu at (131.6, 106.0)
- added R32: 10K, Resistor_SMD:R_0805_2012Metric, F.Cu at (131.6, 102.7)
- added U3: MCP6002-xSN, Package_SO:SOIC-8_3.9x4.9mm_P1.27mm, F.Cu at (158.8, 62.2)
- added U7: LM4562, Package_SO:SOIC-8_3.9x4.9mm_P1.27mm, F.Cu at (138.4, 77.5)
- C10: renamed from C14; value 47nF -> 47n
- C14: renamed from C18; value 47nF -> 47n
- C15: renamed from C19; value 100uF -> 100u
- C20: renamed from C3; value 100nF -> 100n
- C21: renamed from C4; value 100nF -> 100n
- C22: renamed from C5; value 100nF -> 100n
- C23: renamed from C6; value 100nF -> 100n
- C24: renamed from C7; value 1uF -> 1u
- C25: renamed from C8; value 1uF -> 1u
- C26: renamed from C9; value 1uF -> 1u
- C27: renamed from C10; value 1uF -> 1u
- C28: renamed from C11; value 1uF -> 1u
- C29: renamed from C12; value 1uF -> 1u
- C30: renamed from C55; value 100nf -> 100n
- C33: renamed from C35; value 100nF -> 100n
- C34: renamed from C36; value 100nF -> 100n
- C35: renamed from C37; value 100nf -> 100n
- C36: renamed from C38; value 100nF -> 100n
- C49: renamed from C51; value 100nF -> 100n
- C50: renamed from C52; value 100nF -> 100n
- C51: renamed from C53; value 100nF -> 100n
- C52: renamed from C54; value 100nF -> 100n
- R11: renamed from R1; value 82R -> 82
- R16: renamed from R7; value 150R -> 150
- R17: renamed from R8; value 150R -> 150
- U4: renamed from U1; value SN74CBT3253 -> FST5253
- U6: value MCP6002-xSN -> LM4562
- U8: renamed from U9; value SN74CBT3253 -> FST5253
- U9: renamed from U10; value SN74CBT3253 -> FST5253
- moved U6 20.4 mm to (138.4, 61.0)
- moved R11 8.25 mm to (122.6, 86.4), turned to 0 degrees
- moved R30 0.51 mm to (122.6, 88.6)
- renumbered C25 to C1, C15 to C11, C16 to C12, C17 to C13, C20 to C16, C21 to C17, C22 to C18, C2 to C19, C26 to C2, C27 to C3, C33 to C31, C34 to C32, C39 to C37, C40 to C38, C41 to C39, C28 to C4, C42 to C40, C43 to C41, C44 to C42, C45 to C43, C46 to C44, C47 to C45, C48 to C46, C49 to C47, C50 to C48, C29 to C5, C30 to C6, C31 to C7, C32 to C8, C13 to C9, J3 to J2, J2 to J3, R21 to R1, R30 to R10, R3 to R12, R4 to R13, R5 to R14, R6 to R15, R9 to R18, R10 to R19, R22 to R2, R11 to R20, R12 to R21, R13 to R22, R14 to R23, R15 to R24, R16 to R25, R17 to R26, R18 to R27, R19 to R28, R20 to R29, R23 to R3, R31 to R30, R32 to R31, R24 to R4, R25 to R5, R26 to R6, R27 to R7, R28 to R8, R29 to R9, U7 to U1, U8 to U10, U5 to U2, U3 to U5
Connections:
- net 1PPS renamed 1PPS_TEST_SIGNAL
- C11 pad 1: Net-(C15-Pad1) -> Net-(C11-Pad1)
- C12 pad 2: Net-(C15-Pad1) -> Net-(C11-Pad1)
- C16 pad 2: Net-(C20-Pad2) -> Net-(C16-Pad2)
- C17 pad 1: Net-(C20-Pad2) -> Net-(C16-Pad2)
- C26 pad 2: Net-(C9-Pad2) (its old number) -> Net-(C26-Pad2)
- C27 pad 2: Net-(C10-Pad2) -> Net-(C27-Pad2)
- C30 pad 1: RF_OUT -> RF_IN
- J1 pad 16: IR -> Net-(J1-Pad16)
- J1 pad 5: PTT -> Net-(J1-Pad5)
- J3 pad 10: RF_OUT -> RF_IN
- J3 pad 4: BAND_2 -> RF_OUT
- R10 pad 1: Net-(C20-Pad2) -> Net-(C16-Pad2)
- R14 pad 1: Net-(C9-Pad2) (its old number) -> Net-(C26-Pad2)
- R15 pad 2: Net-(C10-Pad2) -> Net-(C27-Pad2)
- R17 pad 1: Net-(R12-Pad1) -> Net-(R17-Pad1)
- R17 pad 2: Net-(R11-Pad1) -> Net-(R17-Pad2)
- R20 pad 1: Net-(R11-Pad1) -> Net-(R17-Pad2)
- R20 pad 2: Net-(R11-Pad2) (its old number) -> Net-(R20-Pad2)
- R21 pad 1: Net-(R12-Pad1) -> Net-(R17-Pad1)
- R21 pad 2: Net-(R12-Pad2) -> Net-(R21-Pad2)
- R24 pad 1: Net-(R11-Pad2) (its old number) -> Net-(R20-Pad2)
- R25 pad 2: Net-(R12-Pad2) -> Net-(R21-Pad2)
- R4 pad 2: Net-(C15-Pad1) -> Net-(C11-Pad1)
- R5 pad 1: Net-(C15-Pad1) -> Net-(C11-Pad1)
- R6 pad 2: Net-(R26-Pad2) -> Net-(R6-Pad2)
- R8 pad 1: Net-(R26-Pad2) -> Net-(R6-Pad2)
- R9 pad 2: Net-(C20-Pad2) -> Net-(C16-Pad2)
- U1 pad 1: Net-(C23-Pad2) -> RX_I
- U1 pad 2: Net-(C24-Pad2) (its old number) -> RX_Q
- U10 pad 1: MIC -> Net-(U10-Pad1)
- U10 pad 19: LO_I -> Net-(C53-Pad1)
- U10 pad 2: LINE_IN -> MIC
- U10 pad 20: LO_Q -> Net-(U10-Pad20)
- U10 pad 21: TRANSMIT_RF -> Net-(U10-Pad21)
- U10 pad 22: PTT -> LO_I
- U10 pad 23: TEST_SIGNAL -> LO_Q
- U10 pad 24: IR -> Net-(U10-Pad24)
- U10 pad 26: +3V3 -> Net-(U10-Pad26)
- U10 pad 6: Net-(U11-Pad5) -> Net-(U10-Pad6)
- U10 pad 7: Net-(U11-Pad6) -> Net-(U10-Pad7)
- U11 pad 5: Net-(U11-Pad5) -> Net-(U10-Pad21)
- U11 pad 6: Net-(U11-Pad6) -> Net-(U10-Pad20)
- U6 pad 1: MIC -> Net-(R21-Pad2)
- U6 pad 2: Net-(R26-Pad2) -> Net-(R17-Pad1)
- U6 pad 3: Net-(C15-Pad1) -> Net-(C27-Pad2)
- U6 pad 5: Net-(C20-Pad2) -> Net-(C26-Pad2)
- U6 pad 6: +2V5 -> Net-(R17-Pad2)
- U6 pad 7: +2V5 -> Net-(R20-Pad2)
- U6 pad 8: +3V3 -> +5V
Routing:
- net GND: track 609.2 -> 99.3 mm, vias 33 -> 23
- net TEST_SIGNAL: track 68.3 -> 0.00 mm, vias 3 -> 0
- net PTT: track 49.3 -> 0.00 mm, vias 1 -> 0
- net Net-(C9-Pad2) (its old number): track 48.0 -> 0.00 mm
- net Net-(U10-Pad20): track 0.00 -> 45.6 mm, vias 0 -> 2
- net +3V3: track 210.7 -> 166.1 mm, vias 7 -> 5
- net Net-(U10-Pad21): track 0.00 -> 42.9 mm, vias 0 -> 2
- net Net-(C26-Pad2): track 0.00 -> 42.2 mm
- net +2V5: track 107.9 -> 147.6 mm, vias 11 -> 8
- net IR: track 39.2 -> 0.00 mm, vias 5 -> 0
- net Net-(J1-Pad5): track 0.00 -> 33.0 mm, vias 0 -> 1
- net TRANSMIT_RF: track 27.9 -> 0.00 mm
- net BAND_2: track 53.6 -> 28.0 mm
- net RF_IN: track 0.00 -> 25.4 mm
- net Net-(U11-Pad5): track 25.1 -> 0.00 mm, vias 1 -> 0
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Other:
- rule trace_min: 0.15 -> 0.16
