File: pcb/openxcvr/RADIO.kicad_pcb (KiCad board)
At the start: 2 copper layers, 99.1 x 99.1 mm, 139 parts, among them J1 Microphone, J2 Mic, J3 Speaker, J4 Headphone, J5 Conn_02x08_Odd_Even, J6 GPS_CONNECTOR, J7 PTT, J8 Conn_01x03_Male, SW1 SW_Push, SW2 SW_Push, SW3 SW_Push, SW4 SW_Push, SW5 Rotary_Encoder_Switch, T1 BN43-2402, U1 PCM1802, U2 TPA711D, U3 MCP6002-xSN, U4 LM4562, U5 FST3253, U6 74CBT3251, U7 74CBT3251, U8 MAX_1000, U9 24LC256

Commit message: Review schematic and PCB layout
Parts:
- added REF**: ESD-Logo_6.6x6mm_SilkScreen, Symbol:ESD-Logo_6.6x6mm_SilkScreen, B.Cu at (95.8, 139.2)
- added REF**: ESD-Logo_6.6x6mm_SilkScreen, Symbol:ESD-Logo_6.6x6mm_SilkScreen, F.Cu at (95.4, 139.2)
- added REF**: OSHW-Logo2_7.3x6mm_SilkScreen, Symbol:OSHW-Logo2_7.3x6mm_SilkScreen, B.Cu at (107.4, 111.8)
- added REF**: OSHW-Logo2_7.3x6mm_SilkScreen, Symbol:OSHW-Logo2_7.3x6mm_SilkScreen, F.Cu at (125.1, 123.1)
- J5: value Conn_02x08_Odd_Even -> TX BOARD CONNECTOR
- J8: value Conn_01x03_Male -> IQ TEST

Commit message: PCB reviewed and updated
Parts:
- added C52: 100n, Capacitor_SMD:C_0805_2012Metric, B.Cu at (99.3, 82.0)
- added C53: 100u, Capacitor_Tantalum_SMD:CP_EIA-7343-31_Kemet-D, F.Cu at (111.0, 69.8)
- added R45: 100K, Resistor_SMD:R_0805_2012Metric, B.Cu at (99.3, 79.9)
- added R46: 100K, Resistor_SMD:R_0805_2012Metric, B.Cu at (103.4, 79.8)
- added R47: 1K, Resistor_SMD:R_0805_2012Metric, B.Cu at (108.2, 66.3)
- moved REF** 8.32 mm to (124.1, 114.8)
- moved J3 4.32 mm to (118.1, 68.5)
- moved REF** 2.90 mm to (93.2, 140.6)
- moved REF** 2.79 mm to (93.0, 140.6)
- moved J2 1.91 mm to (124.3, 68.5)
Connections:
- J3 pad 2: Net-(J3-Pad2) -> Net-(C53-Pad1)
- J4 pad S: Net-(J4-PadS) -> Net-(C53-Pad2)
- J4 pad SN: Net-(J3-Pad1) -> Net-(J4-PadSN)
- J4 pad T: Net-(J4-PadT) -> Net-(C53-Pad2)
- J4 pad TN: Net-(J3-Pad2) -> Net-(J4-PadTN)
- R9 pad 2: Net-(J4-PadT) -> Net-(C53-Pad1)
- U2 pad 3: GND -> Net-(C52-Pad2)
- U2 pad 5: Net-(J4-PadT) -> Net-(C53-Pad1)
- U2 pad 8: Net-(J4-PadS) -> Net-(J3-Pad1)
Routing:
- net Net-(C53-Pad1): track 0.00 -> 43.1 mm, vias 0 -> 2
- net Net-(J4-PadT): track 41.1 -> 0.00 mm
- net Net-(J4-PadTN): track 0.00 -> 31.7 mm, vias 0 -> 3
- net Net-(J4-PadS): track 29.5 -> 0.00 mm
- net Net-(J3-Pad2): track 22.3 -> 0.00 mm
- net Net-(C53-Pad2): track 0.00 -> 21.9 mm, vias 0 -> 1
- net Net-(C52-Pad2): track 0.00 -> 19.1 mm
- net Net-(J3-Pad1): track 12.9 -> 28.4 mm
- net +5VD: track 108.0 -> 109.2 mm
- net Net-(C14-Pad1): track 44.2 -> 45.5 mm
- net +5VA: track 8.37 -> 9.27 mm, vias 0 -> 2
- net Net-(J1-PadTN): track 9.06 -> 9.69 mm
- net GND: track 62.7 -> 63.4 mm, vias 500 -> 489
Other:
- board text added: ".- -... -.-. -.."
- board text added: "Band-Pass Filter"
- board text added: "Microphone Pre Amplifier"
- board text removed: "Band Pass Filter"
- board text removed: "Micorphone Pre Amplifier"

Commit message: move resistors near LCD mounting hole
Parts:
- moved R5 12.7 mm to (99.3, 89.6)
- moved C13 12.7 mm to (99.3, 91.7)
- moved FB2 2.54 mm to (96.5, 73.7), turned to -90 degrees
- moved U2 1.08 mm to (105.4, 87.0)
- moved C10 1.06 mm to (99.3, 87.4)
- moved C15 1.06 mm to (103.4, 83.1)
- moved C52 1.06 mm to (99.3, 83.1)
- moved FB1 1.06 mm to (107.1, 83.1)
- moved R45 1.06 mm to (99.3, 80.9)
- moved R46 1.06 mm to (103.4, 80.8)
- moved R9 1.06 mm to (99.3, 85.3)
Routing:
- net Net-(R5-Pad2): track 14.9 -> 23.5 mm
- net Net-(C53-Pad1): track 43.1 -> 49.2 mm
- net Net-(J4-PadTN): track 31.7 -> 37.8 mm, vias 3 -> 1
- net Net-(C52-Pad2): track 19.1 -> 13.5 mm
- net Net-(C13-Pad1): track 123.9 -> 119.9 mm
- net +5VD: track 109.2 -> 106.0 mm
- net GND: track 63.4 -> 61.1 mm, vias 489 -> 490
- net +5V: track 286.3 -> 287.9 mm
- net +5VA: vias 2 -> 0
- net (no net): vias 0 -> 2
