File: pcb/openxcvr/TX_BOARD.kicad_pcb (KiCad board)
At the start: 2 copper layers, 99.1 x 63.5 mm, 66 parts, among them J1 Power Amplifier, J2 RADIO_CONNECTOR, J3 Antenna, J4 12V_IN, K1 G5V-2, K2 G5V-2, K3 G5V-2, K5 G5V-2, Q1 BS170, Q2 BS170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

Commit message: Candidate design
Parts:
- added R10: 10k, Resistor_SMD:R_0805_2012Metric, B.Cu at (155.6, 101.5)
- added R11: 10k, Resistor_SMD:R_0805_2012Metric, B.Cu at (153.0, 101.6)
- C2, C3, R5, R6: moved to B.Cu
- moved L16 72.3 mm to (130.4, 97.5), turned to 180 degrees
- moved C70 69.6 mm to (130.4, 54.4), turned to 180 degrees
- moved C66 64.1 mm to (130.4, 59.4), turned to 180 degrees
- moved C58 63.9 mm to (130.4, 89.9), turned to 0 degrees
- moved K5 60.6 mm to (188.8, 74.7), turned to 180 degrees
- moved L24 58.4 mm to (130.4, 67.1), turned to 180 degrees
- moved L20 58.2 mm to (130.4, 82.3), turned to 180 degrees
- moved L15 58.0 mm to (140.6, 97.5), turned to 180 degrees
- moved C62 56.3 mm to (130.4, 74.7), turned to 180 degrees
- moved C69 54.4 mm to (140.6, 54.4), turned to 180 degrees
- moved D1 53.5 mm to (185.0, 78.5), turned to 0 degrees
- moved D4 53.0 mm to (185.0, 74.7), turned to 180 degrees
- moved L14 48.1 mm to (150.7, 97.5), turned to 180 degrees
- moved C65 47.3 mm to (140.6, 59.4), turned to 180 degrees
- moved C57 47.0 mm to (140.6, 89.9), turned to 0 degrees
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Connections:
- net VBATT renamed Net-(C2-Pad1)
- C3 pad 1: 5V_OUT -> +5V
- C55 pad 1: LPF_BAND_0_A -> LPF_BAND_3_A
- C56 pad 1: LPF_BAND_1_A -> LPF_BAND_2_A
- C57 pad 1: LPF_BAND_2_A -> LPF_BAND_1_A
- C58 pad 1: LPF_BAND_3_A -> LPF_BAND_0_A
- C67 pad 1: LPF_BAND_0_B -> LPF_BAND_3_B
- C68 pad 1: LPF_BAND_1_B -> LPF_BAND_2_B
- C69 pad 1: LPF_BAND_2_B -> LPF_BAND_1_B
- C70 pad 1: LPF_BAND_3_B -> LPF_BAND_0_B
- J1 pad 2: PA_OUT -> RF_IN
- J2 pad 10: RF_IN -> RF_OUT
- J2 pad 4: BAND_2 -> RF_IN
- J2 pad 7: 5V_OUT -> +5V
- K1 pad 13: RF_IN -> LPF_TXRX
- K1 pad 4: RF_TXRX -> LPF_SWR
- K5 pad 13: PA_OUT -> Net-(K5-Pad13)
- K5 pad 4: ANTENNA -> LPF_TXRX
- K5 pad 6: RF_TXRX -> RF_OUT
- K5 pad 8: RF_OUT -> PA_IN
- K5 pad 9: RF_TXRX -> Net-(K5-Pad9)
- L13 pad 1: LPF_BAND_0_A -> LPF_BAND_3_A
- L14 pad 1: LPF_BAND_1_A -> LPF_BAND_2_A
- L15 pad 1: LPF_BAND_2_A -> LPF_BAND_1_A
- L16 pad 1: LPF_BAND_3_A -> LPF_BAND_0_A
- L21 pad 2: LPF_BAND_0_B -> LPF_BAND_3_B
- L22 pad 2: LPF_BAND_1_B -> LPF_BAND_2_B
- L23 pad 2: LPF_BAND_2_B -> LPF_BAND_1_B
- L24 pad 2: LPF_BAND_3_B -> LPF_BAND_0_B
- TR1 pad 3: PA_IN -> LPF_SWR
- TR1 pad 4: RF_OUT -> ANTENNA
- TR2 pad 2: PA_IN -> LPF_SWR
- U1 pad 3: 5V_OUT -> +5V
Routing:
- net GND: track 499.1 -> 6.33 mm, vias 0 -> 11
- net +5V: track 27.9 -> 177.2 mm, vias 0 -> 1
- net 5V_OUT: track 80.8 -> 0.00 mm
- net Net-(D1-Pad2): track 47.6 -> 121.1 mm
- net PA_IN: track 32.0 -> 88.4 mm
- net Net-(D3-Pad2): track 38.3 -> 91.7 mm
- net RF_TXRX: track 51.7 -> 0.00 mm
- net LPF_BAND_3_B: track 60.3 -> 8.99 mm
- net RF_OUT: track 39.4 -> 79.7 mm
- net LPF_SWR: track 0.00 -> 34.9 mm
- net RF_IN: track 49.0 -> 16.9 mm, vias 1 -> 0
- net LPF_BAND_0_A: track 22.3 -> 54.4 mm
- net LPF_BAND_0_B: track 19.4 -> 51.3 mm
- net LPF_BAND_3_A: track 60.7 -> 29.6 mm
- net PA_OUT: track 30.9 -> 0.00 mm, vias 1 -> 0
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Other:
- board text added: "OpenXCVR 0.1 TX Board JPDawson 2020"
- board text removed: "OpenXCVR TX Board rev 1 JPDawson 2020"
