File: pcb/openxcvr/UI.kicad_pcb (KiCad board)
At the start: 2 copper layers, 99.1 x 63.5 mm, 27 parts, among them J1 UI_CONNECTOR, J2 Mic, J3 Microphone, J4 Speaker, J5 PTT, J6 Headphone, J7 infrared photo module, SW1 SW_Push, SW2 SW_Push, SW3 SW_Push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

Commit message: Candidate design
Parts:
- removed J7: infrared photo module, Connector_PinHeader_2.54mm:PinHeader_1x03_P2.54mm_Vertical
- added R11: 10K, Resistor_SMD:R_0805_2012Metric, F.Cu at (186.9, 96.0)
- added R12: 10K, Resistor_SMD:R_0805_2012Metric, F.Cu at (186.8, 99.3)
- added R13: 10K, Resistor_SMD:R_0805_2012Metric, F.Cu at (186.8, 72.5)
- added R14: 2K2, Resistor_SMD:R_0805_2012Metric, F.Cu at (186.8, 69.8)
- R1, R2, R3, R4: value 10K -> 2K2
- R5: moved to B.Cu
- R6: value 1K -> 2K2
- moved R5 26.4 mm to (180.2, 86.0)
- moved R6 0.51 mm to (180.2, 89.4), turned to 180 degrees
Connections:
- J1 pad 16: IR -> Net-(J1-Pad16)
- J1 pad 5: PTT -> TX_ENABLE
- J5 pad S: PTT -> Net-(J5-PadS)
- J5 pad T: Net-(J5-PadT) -> TX_ENABLE
- R1 pad 1: Net-(R1-Pad1) -> +3V3
- R1 pad 2: GND -> Net-(R1-Pad2)
- R2 pad 1: Net-(R2-Pad1) -> +3V3
- R2 pad 2: GND -> Net-(R2-Pad2)
- R3 pad 1: Net-(R3-Pad1) -> +3V3
- R3 pad 2: GND -> Net-(R3-Pad2)
- R4 pad 1: Net-(R10-Pad2) -> +3V3
- R4 pad 2: GND -> Net-(R10-Pad2)
- R6 pad 2: PTT -> TX_ENABLE
- R7 pad 2: Net-(R1-Pad1) -> Net-(R1-Pad2)
- R8 pad 2: Net-(R2-Pad1) -> Net-(R2-Pad2)
- R9 pad 2: Net-(R3-Pad1) -> Net-(R3-Pad2)
- SW1 pad 1: Net-(R1-Pad1) -> GND
- SW1 pad 2: PB_0 -> Net-(R1-Pad2)
- SW2 pad 1: Net-(R2-Pad1) -> GND
- SW2 pad 2: PB_0 -> Net-(R2-Pad2)
- SW3 pad 1: Net-(R3-Pad1) -> GND
- SW3 pad 2: PB_0 -> Net-(R3-Pad2)
- SW4 pad 1: Net-(R10-Pad2) -> GND
- SW4 pad 2: PB_0 -> Net-(R10-Pad2)
- SW5 pad A: Net-(R1-Pad1) -> PB_1
- SW5 pad B: Net-(R2-Pad1) -> PB_0
- SW5 pad C: PB_1 -> GND
- SW5 pad S1: PB_1 -> SW_SEND
- SW5 pad S2: Net-(R3-Pad1) -> GND
Routing:
- net GND: track 336.1 -> 5.84 mm, vias 4 -> 7
- net +3V3: track 45.1 -> 164.1 mm
- net Net-(R1-Pad1): track 106.1 -> 0.00 mm
- net Net-(R2-Pad1): track 105.0 -> 0.00 mm
- net Net-(R3-Pad1): track 78.5 -> 0.00 mm, vias 1 -> 0
- net TX_ENABLE: track 0.00 -> 59.2 mm
- net PTT: track 58.6 -> 0.00 mm
- net PB_0: track 94.5 -> 36.8 mm
- net IR: track 37.2 -> 0.00 mm, vias 1 -> 0
- net Net-(R1-Pad2): track 0.00 -> 24.2 mm
- net LCD_RS: track 73.9 -> 96.6 mm, vias 4 -> 0
- net PB_1: track 48.5 -> 26.3 mm
- net Net-(R3-Pad2): track 0.00 -> 21.4 mm
- net Net-(R2-Pad2): track 0.00 -> 21.1 mm
- net LCD7: track 57.0 -> 70.7 mm
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Other:
- board text added: "MIC"
- board text added: "OpenXcvr 0.1 UI Board JPDawson 2020"
- board text added: "PTT"
- board text added: "SPK"
