File: pcb/openxcvr/UI.kicad_pcb (KiCad board)
At the start: 2 copper layers, 99.1 x 63.5 mm, 30 parts, among them J1 UI_CONNECTOR, J2 Mic, J3 Microphone, J4 Speaker, J5 PTT, J6 Headphone, SW1 SW_Push, SW2 SW_Push, SW3 SW_Push, SW4 SW_Push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

Commit message: Get things working with rev 1 PCB
Connections:
- J4 pad 1: SPEAKER_HDR -> Net-(J4-Pad1)
- J6 pad TN: Net-(J6-PadTN) -> Net-(J4-Pad1)
Routing:
- net Net-(J4-Pad1): track 0.00 -> 71.9 mm
- net SPEAKER_HDR: track 133.8 -> 148.8 mm
