File: pcb/openxcvr/LPF.sch (KiCad schematic (older format))
At the start: 43 parts, among them J2 RADIO_CONNECTOR, K1 G5V-2, K2 G5V-2, K3 G5V-2, Q1 BS170, Q2 BS170

Commit message: Candidate design
Parts:
- removed J2: RADIO_CONNECTOR, Connector_IDC:IDC-Header_2x05_P2.54mm_Vertical, symbol Connector_Generic:Conn_02x05_Odd_Even
Connections:
- net labels added: LPF_SWR, LPF_TXRX
- net labels removed: 5V_OUT, BAND_2, BATTERY, FWD_PWR, REV_PWR, RF_IN, RF_TXRX, TX_ENABLE
- wire segments 136 -> 125
Other:
- note added: "Fc=14.4MHz (8-16MHz)"
- note added: "Fc=31.66MHz (16-30MHz)"
- note added: "Fc=4.125MHz (2-4MHz)"
- note added: "Fc=7.36MHz (4-8MHz)"
- moved on the sheet: C55, C56, C57, C58, C59, C60, C61, C62, C63, C64, C65, C66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

Commit message: update rev0.2 PCB
Parts:
- renumbered C58 to C1, C65 to C10, C64 to C11, C63 to C12, C70 to C13, C69 to C14, C68 to C15, C67 to C16, C57 to C2, C56 to C3, C55 to C4, C62 to C5, C61 to C6, C60 to C7, C59 to C8, C66 to C9, D4 to D3, L16 to L1, L23 to L10, L22 to L11, L21 to L12, L15 to L2, L14 to L3, L13 to L4, L20 to L5, L19 to L6, L18 to L7, L17 to L8, L24 to L9
Connections:
- net labels added: LPF_ENABLE, PA_OUT, SWR_IN
- net labels removed: +5V, LPF_SWR, LPF_TXRX
- wire segments 125 -> 129

Commit message: Review and update schematic
Other:
- note added: "10T T37-6"
- note added: "11T T37-6"
- note added: "16T T37-6"
- note added: "17T T37-6"
- note added: "19T T37-6"
- note added: "21T T37-6"
- note added: "25T T37-2"
- note added: "27T T37-2"
Changed lines of the file:
@@
 Wire Wire Line
 	9360 5420 9360 5620
+Text Notes 8000 1500 2    50   ~ 0
+10T T37-6
+Text Notes 8000 2700 2    50   ~ 0
+16T T37-6
+Text Notes 8000 3900 2    50   ~ 0
+19T T37-6
+Text Notes 8000 5100 2    50   ~ 0
+25T T37-2
+Text Notes 8600 3900 2    50   ~ 0
+21T T37-6
+Text Notes 8600 5100 2    50   ~ 0
+27T T37-2
+Text Notes 8650 1500 2    50   ~ 0
+11T T37-6
+Text Notes 8650 2700 2    50   ~ 0
+17T T37-6
+Text Notes 9250 1500 2    50   ~ 0
+10T T37-6
+Text Notes 9250 2700 2    50   ~ 0
+16T T37-6
+Text Notes 9250 3900 2    50   ~ 0
+19T T37-6
+Text Notes 9250 5100 2    50   ~ 0
+25T T37-2
 Text Notes 10850 1650 2    50   ~ 0
 Fc=31.66MHz (16-30MHz)

Commit message: Review schematic and PCB layout
Other:
- moved on the sheet: H1, H2, H3, H4
Changed lines of the file:
@@
 $Descr A4 11693 8268
 encoding utf-8
-Sheet 2 4
-Title ""
-Date ""
-Rev ""
-Comp ""
+Sheet 3 4
+Title "Open XCVR"
+Date "2020-06-14"
+Rev "0.2"
+Comp "Jon Dawson"
 Comment1 ""
 Comment2 ""
@@
 Connection ~ 9360 4970
 Wire Wire Line
-	1150 1050 1150 1150
-Wire Wire Line
-	1450 1050 1450 1150
+	1150 850  1150 950
 Wire Wire Line
 	1650 4300 2150 4300
@@
 	1700 5750 2050 5750
 Wire Wire Line
-	1750 1050 1750 1150
-Wire Wire Line
 	1850 2550 2850 2550
 Wire Wire Line
-	2050 1050 2050 1150
+	2000 850  2000 950
 Wire Wire Line
 	2050 3400 2300 3400
@@
 	2800 5700 3150 5700
 Wire Wire Line
+	2850 850  2850 950
+Wire Wire Line
 	2850 1300 2850 2550
 Wire Wire Line
@@
 Wire Wire Line
 	3250 3000 3050 3000
+Wire Wire Line
+	3700 850  3700 950
 Wire Wire Line
 	3700 1700 3950 1700
@@
 L power:GND #PWR01
 U 1 1 5E3CE5BD
-P 1150 1150
-F 0 "#PWR01" H 1150 900 50  0001 C CNN
-F 1 "GND" H 1155 977 50  0000 C CNN
-F 2 "" H 1150 1150 50  0001 C CNN
-F 3 "" H 1150 1150 50  0001 C CNN
-	1    1150 1150
+P 1150 950
+F 0 "#PWR01" H 1150 700 50  0001 C CNN
+F 1 "GND" H 1155 777 50  0000 C CNN
+F 2 "" H 1150 950 50  0001 C CNN
+F 3 "" H 1150 950 50  0001 C CNN
+	1    1150 950
 	1    0    0    -1
 $EndComp
@@
 L power:GND #PWR02
 U 1 1 5E3CEA8A
-P 1450 1150
-F 0 "#PWR02" H 1450 900 50  0001 C CNN
-F 1 "GND" H 1455 977 50  0000 C CNN
-F 2 "" H 1450 1150 50  0001 C CNN
-F 3 "" H 1450 1150 50  0001 C CNN
-	1    1450 1150
-	1    0    0    -1
-$EndComp
-$Comp
-L power:GND #PWR03
-U 1 1 5E3CEEAD
-P 1750 1150
-F 0 "#PWR03" H 1750 900 50  0001 C CNN
-F 1 "GND" H 1755 977 50  0000 C CNN
-F 2 "" H 1750 1150 50  0001 C CNN
-F 3 "" H 1750 1150 50  0001 C CNN
-	1    1750 1150
-	1    0    0    -1
-$EndComp
-$Comp
-L power:GND #PWR04
-U 1 1 5E3CFEDB
-P 2050 1150
-F 0 "#PWR04" H 2050 900 50  0001 C CNN
-F 1 "GND" H 2055 977 50  0000 C CNN
-F 2 "" H 2050 1150 50  0001 C CNN
-F 3 "" H 2050 1150 50  0001 C CNN
-	1    2050 1150
+P 2000 950
+F 0 "#PWR02" H 2000 700 50  0001 C CNN
+F 1 "GND" H 2005 777 50  0000 C CNN
+F 2 "" H 2000 950 50  0001 C CNN
+F 3 "" H 2000 950 50  0001 C CNN
+	1    2000 950
 	1    0    0    -1
 $EndComp
@@
 $EndComp
 $Comp
+L power:GND #PWR03
+U 1 1 5E3CEEAD
+P 2850 950
+F 0 "#PWR03" H 2850 700 50  0001 C CNN
+F 1 "GND" H 2855 777 50  0000 C CNN
+F 2 "" H 2850 950 50  0001 C CNN
+F 3 "" H 2850 950 50  0001 C CNN
+	1    2850 950
+	1    0    0    -1
+$EndComp
+$Comp
 L power:GND #PWR06
 U 1 1 5E478F23
@@
 $EndComp
 $Comp
+L power:GND #PWR04
+U 1 1 5E3CFEDB
+P 3700 950
+F 0 "#PWR04" H 3700 700 50  0001 C CNN
+F 1 "GND" H 3705 777 50  0000 C CNN
+F 2 "" H 3700 950 50  0001 C CNN
+F 3 "" H 3700 950 50  0001 C CNN
+	1    3700 950
+	1    0    0    -1
+$EndComp
+$Comp
 L power:GND #PWR07
 U 1 1 5E520825
@@
 L Mechanical:MountingHole_Pad H1
 U 1 1 5E3C8D4A
-P 1150 950
-F 0 "H1" H 1250 999 50  0000 L CNN
-F 1 "MountingHole_Pad" H 1250 908 50  0000 L CNN
-F 2 "MountingHole:MountingHole_3.2mm_M3_Pad" H 1150 950 50  0001 C CNN
-F 3 "~" H 1150 950 50  0001 C CNN
-	1    1150 950
+P 1150 750
+F 0 "H1" H 1250 799 50  0000 L CNN
+F 1 "MountingHole_Pad" H 1250 708 50  0000 L CNN
+F 2 "MountingHole:MountingHole_3.2mm_M3_Pad" H 1150 750 50  0001 C CNN
+F 3 "~" H 1150 750 50  0001 C CNN
+	1    1150 750
 	1    0    0    -1
 $EndComp
@@
 L Mechanical:MountingHole_Pad H2
 U 1 1 5E3C9BDE
-P 1450 950
-F 0 "H2" H 1550 999 50  0000 L CNN
-F 1 "MountingHole_Pad" H 1550 908 50  0000 L CNN
-F 2 "MountingHole:MountingHole_3.2mm_M3_Pad" H 1450 950 50  0001 C CNN
-F 3 "~" H 1450 950 50  0001 C CNN
-	1    1450 950
+P 2000 750
+F 0 "H2" H 2100 799 50  0000 L CNN
+F 1 "MountingHole_Pad" H 2100 708 50  0000 L CNN
+F 2 "MountingHole:MountingHole_3.2mm_M3_Pad" H 2000 750 50  0001 C CNN
+F 3 "~" H 2000 750 50  0001 C CNN
+	1    2000 750
 	1    0    0    -1
 $EndComp
@@
 L Mechanical:MountingHole_Pad H3
 U 1 1 5E3CC23B
-P 1750 950
-F 0 "H3" H 1850 999 50  0000 L CNN
-F 1 "MountingHole_Pad" H 1850 908 50  0000 L CNN
-F 2 "MountingHole:MountingHole_3.2mm_M3_Pad" H 1750 950 50  0001 C CNN
-F 3 "~" H 1750 950 50  0001 C CNN
-	1    1750 950
+P 2850 750
+F 0 "H3" H 2950 799 50  0000 L CNN
+F 1 "MountingHole_Pad" H 2950 708 50  0000 L CNN
+F 2 "MountingHole:MountingHole_3.2mm_M3_Pad" H 2850 750 50  0001 C CNN
+F 3 "~" H 2850 750 50  0001 C CNN
+	1    2850 750
 	1    0    0    -1
 $EndComp
@@
 L Mechanical:MountingHole_Pad H4
 U 1 1 5E3CDA31
-P 2050 950
-F 0 "H4" H 2150 999 50  0000 L CNN
-F 1 "MountingHole_Pad" H 2150 908 50  0000 L CNN
-F 2 "MountingHole:MountingHole_3.2mm_M3_Pad" H 2050 950 50  0001 C CNN
-F 3 "~" H 2050 950 50  0001 C CNN
-	1    2050 950
-	1    0    0    -1
-$EndComp
+P 3700 750
+F 0 "H4" H 3800 799 50  0000 L CNN
+F 1 "MountingHole_Pad" H 3800 708 50  0000 L CNN
+F 2 "MountingHole:MountingHole_3.2mm_M3_Pad" H 3700 750 50  0001 C CNN
+F 3 "~" H 3700 750 50  0001 C CNN
+	1    3700 750
+	1    0    0    -1
+$EndComp
