File: pcb/openxcvr/MAX1000.sch (KiCad schematic (older format))
At the start: 11 parts, among them J1 UI_CONNECTOR, J2 PA_CONNECTOR, J3 GPS_CONNECTOR, J4 TEST_SIGNAL_CONNECTOR, U11 24LC256, U8 MAX_1000

Commit message: Candidate design
Parts:
- removed J4: TEST_SIGNAL_CONNECTOR, Connector_PinHeader_2.54mm:PinHeader_1x02_P2.54mm_Vertical, symbol Connector:Conn_01x02_Male
- added C53: 100n, Capacitor_SMD:C_0805_2012Metric, symbol Device:C
- added R32: 10K, Resistor_SMD:R_0805_2012Metric, symbol Device:R
- renumbered J3 to J2, J2 to J3, U8 to U10
Connections:
- net labels added: 1PPS_TEST_SIGNAL, RF_IN
- net labels removed: 1PPS, IR, PTT, TEST_SIGNAL, TRANSMIT_RF
- wire segments 107 -> 96
- no-connect marks 6 -> 11
Other:
- moved on the sheet: H1, H2, H3, H4, J2

Commit message: Get things working with rev 1 PCB
Parts:
- RV3: footprint Potentiometer_THT:Potentiometer_Piher_PT-6-V_Vertical -> Potentiometer_THT:Potentiometer_Piher_PT-6-H_Horizontal
Changed lines of the file:
@@
 NoConn ~ 3100 4650
 NoConn ~ 5250 1950
-NoConn ~ 6400 2350
 NoConn ~ 5250 2450
 NoConn ~ 5250 2550
 NoConn ~ 5250 2650
 NoConn ~ 6400 2150
+NoConn ~ 6400 2350
 Wire Wire Line
 	1000 950  1000 1050
@@
 F 0 "RV3" H 2380 5745 50  0000 R CNN
 F 1 "10K" H 2380 5655 50  0000 R CNN
-F 2 "Potentiometer_THT:Potentiometer_Piher_PT-6-V_Vertical" H 2450 5700 50  0001 C CNN
+F 2 "Potentiometer_THT:Potentiometer_Piher_PT-6-H_Horizontal" H 2450 5700 50  0001 C CNN
 F 3 "~" H 2450 5700 50  0001 C CNN
 	1    2450 5700

Commit message: Add eeprom load store capability
Parts:
- removed J1: UI_CONNECTOR, Connector_IDC:IDC-Header_2x10_P2.54mm_Vertical, symbol Connector_Generic:Conn_02x10_Odd_Even
- removed R32: 10K, Resistor_SMD:R_0805_2012Metric, symbol Device:R
- removed RV3: 10K, Potentiometer_THT:Potentiometer_Piher_PT-6-H_Horizontal, symbol Device:R_POT_TRIM
- added FB1, FB2, FB3: Ferrite_Bead, Inductor_SMD:L_0805_2012Metric, symbol Device:Ferrite_Bead
- added R21, R22, R23, R24, R25, R26, R27, R28: 100, Resistor_SMD:R_0805_2012Metric, symbol Device:R
- renumbered C53 to C50, J3 to J5, J2 to J6, U10 to U8, U11 to U9
Connections:
- net labels added: +5VA, +5VD, DAH, DIT, PTT
- net labels removed: LCD_CONTRAST, MIC_HDR, SPEAKER_HDR
- wire segments 96 -> 95
- no-connect marks 11 -> 3
Other:
- note added: "Seperate supply for analogue"
- note added: "Seperate supply for audio amplifier"
- moved on the sheet: J6

Commit message: update rev0.2 PCB
Parts:
- removed C50: 100n, Capacitor_SMD:C_0805_2012Metric, symbol Device:C
- removed J5: PA_CONNECTOR, Connector_IDC:IDC-Header_2x05_P2.54mm_Vertical, symbol Connector_Generic:Conn_02x05_Odd_Even
- added J5: Conn_02x08_Odd_Even, Connector_PinHeader_2.54mm:PinHeader_2x08_P2.54mm_Vertical, symbol Connector_Generic:Conn_02x08_Odd_Even
- U8: symbol xcvr_components:MAX_1000 -> RADIO-rescue:MAX_1000-xcvr_components
Connections:
- wire segments 95 -> 105
Changed lines of the file:
@@
 Comment9 ""
 $EndDescr
+Connection ~ 2650 5000
+Connection ~ 3500 4800
+Connection ~ 3500 4900
 Connection ~ 6500 4600
 Connection ~ 6700 1100
@@
 	1900 950  1900 1050
 Wire Wire Line
-	2550 5450 2850 5450
-Wire Wire Line
-	2550 5550 2850 5550
-Wire Wire Line
-	2550 5650 2850 5650
-Wire Wire Line
-	2550 5750 2850 5750
-Wire Wire Line
-	2700 5850 2850 5850
-Wire Wire Line
-	2700 5950 2700 5850
+	2550 4200 2850 4200
+Wire Wire Line
+	2550 4300 2850 4300
+Wire Wire Line
+	2550 4400 2850 4400
+Wire Wire Line
+	2550 4500 2850 4500
+Wire Wire Line
+	2650 4900 2850 4900
+Wire Wire Line
+	2650 5000 2650 4900
+Wire Wire Line
+	2650 5000 3500 5000
+Wire Wire Line
+	2650 5150 2650 5000
 Wire Wire Line
 	2800 950  2800 1050
 Wire Wire Line
+	2850 4600 2550 4600
+Wire Wire Line
+	2850 4700 2550 4700
+Wire Wire Line
+	2850 4800 2550 4800
+Wire Wire Line
 	3050 6600 3550 6600
 Wire Wire Line
 	3300 6700 3300 6750
 Wire Wire Line
-	3350 5450 3950 5450
-Wire Wire Line
-	3350 5550 3950 5550
-Wire Wire Line
-	3350 5650 3950 5650
-Wire Wire Line
-	3350 5750 3950 5750
-Wire Wire Line
-	3350 5850 3950 5850
+	3350 4200 3950 4200
+Wire Wire Line
+	3350 4300 3950 4300
+Wire Wire Line
+	3350 4400 3950 4400
+Wire Wire Line
+	3350 4500 3950 4500
+Wire Wire Line
+	3350 4600 3950 4600
+Wire Wire Line
+	3350 4700 3500 4700
+Wire Wire Line
+	3350 4800 3500 4800
+Wire Wire Line
+	3350 4900 3500 4900
+Wire Wire Line
+	3500 4700 3500 4800
+Wire Wire Line
+	3500 4800 3500 4900
+Wire Wire Line
+	3500 5000 3500 4900
 Wire Wire Line
 	3550 6700 3300 6700
@@
 	6400 2750 8850 2750
 Wire Wire Line
-	6400 2850 7400 2850
+	6400 2850 7000 2850
 Wire Wire Line
 	6400 2950 7000 2950
@@
 Wire Wire Line
 	7700 1750 7700 1600
-Wire Wire Line
-	7700 2850 7900 2850
 Wire Wire Line
 	8600 2850 8600 3150
@@
 Text Notes 9250 950  2    50   ~ 0
 Seperate supply for audio amplifier
-Text GLabel 2550 5450 0    50   Input ~ 0
+Text GLabel 2550 4200 0    50   Input ~ 0
 BATTERY
-Text GLabel 2550 5550 0    50   Input ~ 0
+Text GLabel 2550 4300 0    50   Input ~ 0
 FWD_PWR
-Text GLabel 2550 5650 0    50   Input ~ 0
+Text GLabel 2550 4400 0    50   Input ~ 0
 REV_PWR
-Text GLabel 2550 5750 0    50   Output ~ 0
+Text GLabel 2550 4500 0    50   Output ~ 0
 5V_IN
+Text GLabel 2550 4600 0    50   Output ~ 0
+RF_OUT
+Text GLabel 2550 4700 0    50   Output ~ 0
+LO_Q
+Text GLabel 2550 4800 0    50   Output ~ 0
+LO_I
 Text GLabel 3050 6600 0    50   BiDi ~ 0
 1PPS_TEST_SIGNAL
-Text GLabel 3950 5450 2    50   BiDi ~ 0
+Text GLabel 3950 4200 2    50   BiDi ~ 0
 TX_ENABLE
-Text GLabel 3950 5550 2    50   Output ~ 0
-RF_OUT
-Text GLabel 3950 5650 2    50   Output ~ 0
+Text GLabel 3950 4300 2    50   Output ~ 0
+BAND_2
+Text GLabel 3950 4400 2    50   Output ~ 0
 BAND_1
-Text GLabel 3950 5750 2    50   Output ~ 0
+Text GLabel 3950 4500 2    50   Output ~ 0
 BAND_0
-Text GLabel 3950 5850 2    50   Input ~ 0
+Text GLabel 3950 4600 2    50   Input ~ 0
 RF_IN
 Text GLabel 4200 3550 0    50   Input ~ 0
@@
 Text GLabel 7000 2550 2    50   Output ~ 0
 LO_I
+Text GLabel 7000 2850 2    50   Output ~ 0
+RF_OUT
 Text GLabel 7000 2950 2    50   BiDi ~ 0
 TX_ENABLE
@@
 Text GLabel 7350 3850 2    50   Input ~ 0
 PB_0
-Text GLabel 7900 2850 2    50   Output ~ 0
-RF_OUT
 $Comp
 L power:+5VD #PWR073
@@
 L power:GND #PWR068
 U 1 1 5E3AEBD5
-P 2700 5950
-F 0 "#PWR068" H 2700 5700 50  0001 C CNN
-F 1 "GND" H 2705 5777 50  0000 C CNN
-F 2 "" H 2700 5950 50  0001 C CNN
-F 3 "" H 2700 5950 50  0001 C CNN
-	1    2700 5950
+P 2650 5150
+F 0 "#PWR068" H 2650 4900 50  0001 C CNN
+F 1 "GND" H 2655 4977 50  0000 C CNN
+F 2 "" H 2650 5150 50  0001 C CNN
+F 3 "" H 2650 5150 50  0001 C CNN
+	1    2650 5150
 	1    0    0    -1
 $EndComp
@@
 $EndComp
 $Comp
-L Device:C C50
-U 1 1 5E4FFC23
-P 7550 2850
-F 0 "C50" V 7801 2850 50  0000 C CNN
-F 1 "100n" V 7710 2850 50  0000 C CNN
-F 2 "Capacitor_SMD:C_0805_2012Metric" H 7588 2700 50  0001 C CNN
-F 3 "~" H 7550 2850 50  0001 C CNN
-	1    7550 2850
-	0    -1   -1   0
-$EndComp
-$Comp
 L Device:Ferrite_Bead FB1
 U 1 1 5EA397AC
@@
 $EndComp
 $Comp
-L Connector_Generic:Conn_02x05_Odd_Even J5
-U 1 1 5E38CD1E
-P 3050 5650
-F 0 "J5" H 3100 6066 50  0000 C CNN
-F 1 "PA_CONNECTOR" H 3100 5975 50  0000 C CNN
-F 2 "Connector_IDC:IDC-Header_2x05_P2.54mm_Vertical" H 3050 5650 50  0001 C CNN
-F 3 "~" H 3050 5650 50  0001 C CNN
-	1    3050 5650
+L Connector_Generic:Conn_02x08_Odd_Even J5
+U 1 1 5ECB3DCF
+P 3050 4500
+F 0 "J5" H 3100 5016 50  0000 C CNN
+F 1 "Conn_02x08_Odd_Even" H 3100 4925 50  0000 C CNN
+F 2 "Connector_PinHeader_2.54mm:PinHeader_2x08_P2.54mm_Vertical" H 3050 4500 50  0001 C CNN
+F 3 "~" H 3050 4500 50  0001 C CNN
+	1    3050 4500
 	1    0    0    -1
 $EndComp
@@
 $EndComp
 $Comp
-L xcvr_components:MAX_1000 U8
+L RADIO-rescue:MAX_1000-xcvr_components U8
 U 1 1 5E2CD29F
 P 5800 1800

Commit message: Review and update schematic
Parts:
- added C16: 100n, Capacitor_SMD:C_0805_2012Metric, symbol Device:C
- added R43, R44: 0, Resistor_SMD:R_0805_2012Metric, symbol Device:R
Connections:
- wire segments 105 -> 113
Other:
- note added: "Fit for USB power option"
- note added: "Fit for external power only"
- moved on the sheet: FB1, FB2, FB3, J5, J6, R21, R22, R23, R24, R25, R26, R27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

Commit message: Review schematic and PCB layout
Parts:
- J5: value Conn_02x08_Odd_Even -> TX BOARD CONNECTOR
Connections:
- wire segments 113 -> 112
Other:
- moved on the sheet: C16, FB1, FB2, FB3, J5, J6, R21, R22, R23, R24, R25, R26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
