File: pcb/openxcvr/TX_BOARD.sch (KiCad schematic (older format))
At the start: 0 parts

Commit message: update rev0.2 PCB
Changed lines of the file:
@@
 $Descr A4 11693 8268
 encoding utf-8
-Sheet 1 3
+Sheet 1 4
 Title "Open XCVR"
 Date "2020-01-26"
@@
 F1 "TX_RX.sch" 50
 $EndSheet
+$Sheet
+S 7150 2050 2600 900
+U 5EBEA4A7
+F0 "tx_oa" 50
+F1 "tx_pa.sch" 50
+$EndSheet
 $EndSCHEMATC

Commit message: Review and update schematic
Changed lines of the file:
@@
+$EndSheet
+$Sheet
+S 7150 2050 2600 900
+U 5EBEA4A7
+F0 "TX_PA" 50
+F1 "tx_pa.sch" 50
 $EndSheet
 $Sheet
@@
 F1 "TX_RX.sch" 50
 $EndSheet
-$Sheet
-S 7150 2050 2600 900
-U 5EBEA4A7
-F0 "tx_oa" 50
-F1 "tx_pa.sch" 50
-$EndSheet
 $EndSCHEMATC

Commit message: Review schematic and PCB layout
Changed lines of the file:
@@
 Sheet 1 4
 Title "Open XCVR"
-Date "2020-01-26"
-Rev "0.1"
+Date "2020-06-14"
+Rev "0.2"
 Comp "Jon Dawson"
 Comment1 ""
@@
 S 4350 2050 2550 900
 U 5E3F7669
-F0 "LPF" 50
+F0 "low pass filters" 50
 F1 "LPF.sch" 50
 $EndSheet
@@
 S 7150 2050 2600 900
 U 5EBEA4A7
-F0 "TX_PA" 50
+F0 "transmit power amplifier" 50
 F1 "tx_pa.sch" 50
 $EndSheet
@@
 S 4360 3290 2530 950
 U 5E5B8C32
-F0 "TX_RX" 50
+F0 "transmit receive switching " 50
 F1 "TX_RX.sch" 50
 $EndSheet
