File: pcb/openxcvr/TX_RX.sch (KiCad schematic (older format))
At the start: 23 parts, among them J1 Power Amplifier, J3 Antenna, J4 12V_IN, K5 G5V-2, Q3 BS170, Q4 BS170, U1 LM7805_TO220

Commit message: Candidate design
Parts:
- added J2: RADIO_CONNECTOR, Connector_IDC:IDC-Header_2x05_P2.54mm_Vertical, symbol Connector_Generic:Conn_02x05_Odd_Even
- added R10, R11: 10k, Resistor_SMD:R_0805_2012Metric, symbol Device:R
Connections:
- net labels added: BAND_0, BAND_1, LPF_SWR, LPF_TXRX, RF_IN
- net labels removed: 5V_OUT, PA_OUT, RF_TXRX, VBATT
- wire segments 101 -> 117
- no-connect marks 0 -> 3
Other:
- moved on the sheet: C1, C4

Commit message: update rev0.2 PCB
Parts:
- removed D3: 1N4148W, Diode_SMD:D_SOD-123, symbol Diode:1N4148W
- removed J1: Power Amplifier, Connector_PinHeader_2.54mm:PinHeader_1x04_P2.54mm_Vertical, symbol Connector:Conn_01x04_Male
- removed J2: RADIO_CONNECTOR, Connector_IDC:IDC-Header_2x05_P2.54mm_Vertical, symbol Connector_Generic:Conn_02x05_Odd_Even
- removed J3: Antenna, Connector_PinHeader_2.54mm:PinHeader_1x02_P2.54mm_Vertical, symbol Connector:Conn_01x02_Male
- removed J4: 12V_IN, Connector_PinHeader_2.54mm:PinHeader_1x02_P2.54mm_Vertical, symbol Connector:Conn_01x02_Male
- removed K5: G5V-2, Relay_THT:Relay_DPDT_Omron_G5V-2, symbol Relay:G5V-2
- removed Q4: BS170, Package_TO_SOT_THT:TO-92_Inline, symbol Transistor_FET:BS170
- added D4: 1N4148W, Diode_SMD:D_SOD-123, symbol Diode:1N4148W
- added J1: Conn_Coaxial, Connector_Coaxial:BNC_Amphenol_B6252HB-NPP3G-50_Horizontal, symbol Connector:Conn_Coaxial
- added J2: Conn_02x08_Odd_Even, Connector_PinHeader_2.54mm:PinHeader_2x08_P2.54mm_Vertical, symbol Connector_Generic:Conn_02x08_Odd_Even
- added J3: Barrel_Jack_Switch, Connector_BarrelJack:BarrelJack_Horizontal, symbol Connector:Barrel_Jack_Switch
- added K4: G5V-2, Relay_THT:Relay_DPDT_Omron_G5V-2, symbol Relay:G5V-2
- added R13, R4: 10k, Resistor_SMD:R_0805_2012Metric, symbol Device:R
- added U2, U3: to220heatsink, openxcvr:to220 heatsink, symbol xcvr_components:to220heatsink
- TR1, TR2: symbol xcvr_components:FT50-43Transformer -> TX_BOARD-rescue:FT50-43Transformer-xcvr_components
- U1: footprint Package_TO_SOT_THT:TO-220-3_Horizontal_TabDown -> Package_TO_SOT_THT:TO-220-3_Vertical
- renumbered C1 to C17, C2 to C18, C3 to C19, C4 to C20, R8 to R10, R9 to R11, R11 to R12, R10 to R5, R4 to R6, R5 to R7, R6 to R8, R7 to R9
Connections:
- net labels added: +12V, BAND_2, LO_I, LO_Q, LPF_ENABLE, RF_ENVELOPE, SWR_IN
- net labels removed: LPF_SWR, LPF_TXRX, PA_IN, RF_IN, TX_N
- wire segments 117 -> 129
- no-connect marks 3 -> 0
Other:
- moved on the sheet: R3

Commit message: Review and update schematic
Parts:
- added J4: Battery Connector, Connector_PinHeader_2.54mm:PinHeader_1x02_P2.54mm_Vertical, symbol Connector:Conn_01x02_Male
- added SW1: POWER SWITCH, openxcvr:RS PCB Toggle Switch, symbol Switch:SW_SPDT
- J2: value Conn_02x08_Odd_Even -> RADIO BOARD CONNECTOR
- J3: value Barrel_Jack_Switch -> Power Jack
- U1: value LM7805_TO220 -> LM7805CV_TO220
Connections:
- net labels removed: BAND_2, LO_Q
- wire segments 129 -> 133
- no-connect marks 0 -> 4
Other:
- moved on the sheet: J2, R10, R4, R9, U3

Commit message: Review schematic and PCB layout
Parts:
- J1: value Conn_Coaxial -> Antenna BNC Connector
Connections:
- net labels added: VBATT
- net labels removed: BATTERY
Other:
- note added: "Linear Regulator"
- note added: "SWR Bridge"
- note added: "TX RX Switching"
- moved on the sheet: C17, C19, C20, J1, J2, J3, J4, K4, R10, R11, R12, R13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
