File: pcb/openxcvr/adc.sch (KiCad schematic (older format))
At the start: 11 parts, among them U7 PCM1802

Commit message: Candidate design
Parts:
- removed C23, C24: 1u, Capacitor_SMD:C_0805_2012Metric, symbol Device:C
- renumbered C25 to C1, C26 to C2, C27 to C3, C28 to C4, C29 to C5, C30 to C6, C31 to C7, C32 to C8, U7 to U1
Connections:
- wire segments 58 -> 52

Commit message: Get things working with rev 1 PCB
Parts:
- added R12: 1K, Resistor_SMD:R_0805_2012Metric, symbol Device:R
Connections:
- wire segments 52 -> 55
Changed lines of the file:
@@
 Comment9 ""
 $EndDescr
+Connection ~ 4050 3150
 Connection ~ 4050 6150
 Connection ~ 4300 4250
+Connection ~ 4750 3150
 Connection ~ 4750 4250
 Connection ~ 4900 6150
@@
 	3600 3350 3600 3850
 Wire Wire Line
+	3900 2650 3900 3450
+Wire Wire Line
 	3900 6150 4050 6150
 Wire Wire Line
@@
 	3950 4550 3950 4650
 Wire Wire Line
+	4050 3150 4050 2650
+Wire Wire Line
+	4050 3150 4350 3150
+Wire Wire Line
+	4050 3250 4050 3150
+Wire Wire Line
 	4050 6000 4050 6150
 Wire Wire Line
@@
 	4300 4550 4300 4650
 Wire Wire Line
-	4450 2650 4450 3450
-Wire Wire Line
-	4600 3250 4600 2650
+	4650 3150 4750 3150
 Wire Wire Line
 	4750 3150 4750 4250
@@
 	5050 3150 4750 3150
 Wire Wire Line
-	5050 3250 4600 3250
+	5050 3250 4050 3250
 Wire Wire Line
 	5050 3350 3600 3350
 Wire Wire Line
-	5050 3450 4450 3450
+	5050 3450 3900 3450
 Wire Wire Line
 	5050 3750 4950 3750
@@
 LRCK
 $Comp
+L power:+3V3 #PWR07
+U 1 1 5E38F1B7
+P 3900 2650
+F 0 "#PWR07" H 3900 2500 50  0001 C CNN
+F 1 "+3V3" H 3915 2823 50  0000 C CNN
+F 2 "" H 3900 2650 50  0001 C CNN
+F 3 "" H 3900 2650 50  0001 C CNN
+	1    3900 2650
+	1    0    0    -1
+$EndComp
+$Comp
+L power:+5V #PWR08
+U 1 1 5E38C061
+P 4050 2650
+F 0 "#PWR08" H 4050 2500 50  0001 C CNN
+F 1 "+5V" H 4065 2823 50  0000 C CNN
+F 2 "" H 4050 2650 50  0001 C CNN
+F 3 "" H 4050 2650 50  0001 C CNN
+	1    4050 2650
+	1    0    0    -1
+$EndComp
+$Comp
 L power:+3V3 #PWR04
 U 1 1 5E38CACB
@@
 F 3 "" H 4050 6000 50  0001 C CNN
 	1    4050 6000
-	1    0    0    -1
-$EndComp
-$Comp
-L power:+3V3 #PWR07
-U 1 1 5E38F1B7
-P 4450 2650
-F 0 "#PWR07" H 4450 2500 50  0001 C CNN
-F 1 "+3V3" H 4465 2823 50  0000 C CNN
-F 2 "" H 4450 2650 50  0001 C CNN
-F 3 "" H 4450 2650 50  0001 C CNN
-	1    4450 2650
-	1    0    0    -1
-$EndComp
-$Comp
-L power:+5V #PWR08
-U 1 1 5E38C061
-P 4600 2650
-F 0 "#PWR08" H 4600 2500 50  0001 C CNN
-F 1 "+5V" H 4615 2823 50  0000 C CNN
-F 2 "" H 4600 2650 50  0001 C CNN
-F 3 "" H 4600 2650 50  0001 C CNN
-	1    4600 2650
 	1    0    0    -1
 $EndComp
@@
 $EndComp
 $Comp
+L Device:R R12
+U 1 1 5E61E083
+P 4500 3150
+F 0 "R12" V 4706 3150 50  0000 C CNN
+F 1 "1K" V 4615 3150 50  0000 C CNN
+F 2 "Resistor_SMD:R_0805_2012Metric" V 4430 3150 50  0001 C CNN
+F 3 "~" H 4500 3150 50  0001 C CNN
+	1    4500 3150
+	0    -1   -1   0
+$EndComp
+$Comp

Commit message: Add eeprom load store capability
Parts:
- renumbered R12 to R1
Changed lines of the file:
@@
 $Descr A4 11693 8268
 encoding utf-8
-Sheet 2 6
+Sheet 2 7
 Title "Open XCVR"
 Date "2020-01-26"
@@
 LRCK
 $Comp
-L power:+3V3 #PWR07
+L power:+3V3 #PWR02
 U 1 1 5E38F1B7
 P 3900 2650
-F 0 "#PWR07" H 3900 2500 50  0001 C CNN
+F 0 "#PWR02" H 3900 2500 50  0001 C CNN
 F 1 "+3V3" H 3915 2823 50  0000 C CNN
 F 2 "" H 3900 2650 50  0001 C CNN
@@
 $EndComp
 $Comp
-L power:+5V #PWR08
+L power:+5V #PWR05
 U 1 1 5E38C061
 P 4050 2650
-F 0 "#PWR08" H 4050 2500 50  0001 C CNN
+F 0 "#PWR05" H 4050 2500 50  0001 C CNN
 F 1 "+5V" H 4065 2823 50  0000 C CNN
 F 2 "" H 4050 2650 50  0001 C CNN
@@
 $EndComp
 $Comp
-L power:+3V3 #PWR04
+L power:+3V3 #PWR06
 U 1 1 5E38CACB
 P 4050 6000
-F 0 "#PWR04" H 4050 5850 50  0001 C CNN
+F 0 "#PWR06" H 4050 5850 50  0001 C CNN
 F 1 "+3V3" H 4065 6173 50  0000 C CNN
 F 2 "" H 4050 6000 50  0001 C CNN
@@
 $EndComp
 $Comp
-L power:GND #PWR02
+L power:GND #PWR03
 U 1 1 5E3EBF7E
 P 3900 6550
-F 0 "#PWR02" H 3900 6300 50  0001 C CNN
+F 0 "#PWR03" H 3900 6300 50  0001 C CNN
 F 1 "GND" H 3905 6377 50  0000 C CNN
 F 2 "" H 3900 6550 50  0001 C CNN
@@
 $EndComp
 $Comp
-L power:GND #PWR03
+L power:GND #PWR04
 U 1 1 5E3E42CA
 P 3950 4650
-F 0 "#PWR03" H 3950 4400 50  0001 C CNN
+F 0 "#PWR04" H 3950 4400 50  0001 C CNN
 F 1 "GND" H 3955 4477 50  0000 C CNN
 F 2 "" H 3950 4650 50  0001 C CNN
@@
 $EndComp
 $Comp
-L power:GND #PWR05
+L power:GND #PWR07
 U 1 1 5E3EBFB7
 P 4250 6550
-F 0 "#PWR05" H 4250 6300 50  0001 C CNN
+F 0 "#PWR07" H 4250 6300 50  0001 C CNN
 F 1 "GND" H 4255 6377 50  0000 C CNN
 F 2 "" H 4250 6550 50  0001 C CNN
@@
 $EndComp
 $Comp
-L power:GND #PWR06
+L power:GND #PWR08
 U 1 1 5E3E48F2
 P 4300 4650
-F 0 "#PWR06" H 4300 4400 50  0001 C CNN
+F 0 "#PWR08" H 4300 4400 50  0001 C CNN
 F 1 "GND" H 4305 4477 50  0000 C CNN
 F 2 "" H 4300 4650 50  0001 C CNN
@@
 $EndComp
 $Comp
-L Device:R R12
+L Device:R R1
 U 1 1 5E61E083
 P 4500 3150
-F 0 "R12" V 4706 3150 50  0000 C CNN
+F 0 "R1" V 4706 3150 50  0000 C CNN
 F 1 "1K" V 4615 3150 50  0000 C CNN
 F 2 "Resistor_SMD:R_0805_2012Metric" V 4430 3150 50  0001 C CNN

Commit message: update rev0.2 PCB
Parts:
- U1: symbol xcvr_components:PCM1802 -> RADIO-rescue:PCM1802-xcvr_components
Changed lines of the file:
@@
 $EndComp
 $Comp
-L xcvr_components:PCM1802 U1
+L RADIO-rescue:PCM1802-xcvr_components U1
 U 1 1 5E385964
 P 5750 3300

Commit message: Review schematic and PCB layout
Other:
- moved on the sheet: R1
Changed lines of the file:
@@
 Sheet 2 7
 Title "Open XCVR"
-Date "2020-01-26"
-Rev "0.1"
+Date "2020-06-14"
+Rev "0.2"
 Comp "Jon Dawson"
 Comment1 ""
@@
 Comment9 ""
 $EndDescr
-Connection ~ 4050 3150
+Connection ~ 3550 3150
 Connection ~ 4050 6150
 Connection ~ 4300 4250
@@
 NoConn ~ 5050 3650
 Wire Wire Line
-	3400 2850 5050 2850
-Wire Wire Line
-	3400 2950 5050 2950
-Wire Wire Line
-	3600 3350 3600 3850
-Wire Wire Line
-	3900 2650 3900 3450
+	3100 3350 3100 3850
+Wire Wire Line
+	3350 2650 3350 3450
+Wire Wire Line
+	3550 3150 3550 2650
+Wire Wire Line
+	3550 3150 3850 3150
+Wire Wire Line
+	3550 3250 3550 3150
 Wire Wire Line
 	3900 6150 4050 6150
@@
 	3950 4550 3950 4650
 Wire Wire Line
-	4050 3150 4050 2650
-Wire Wire Line
-	4050 3150 4350 3150
-Wire Wire Line
-	4050 3250 4050 3150
-Wire Wire Line
 	4050 6000 4050 6150
 Wire Wire Line
 	4050 6150 4250 6150
 Wire Wire Line
+	4150 3150 4750 3150
+Wire Wire Line
 	4250 6450 4250 6550
 Wire Wire Line
@@
 	4300 4550 4300 4650
 Wire Wire Line
-	4650 3150 4750 3150
+	4700 2800 2700 2800
+Wire Wire Line
+	4700 2950 4700 2800
+Wire Wire Line
+	4750 2700 2700 2700
+Wire Wire Line
+	4750 2850 4750 2700
 Wire Wire Line
 	4750 3150 4750 4250
@@
 	4950 3850 7150 3850
 Wire Wire Line
+	5050 2850 4750 2850
+Wire Wire Line
+	5050 2950 4700 2950
+Wire Wire Line
 	5050 3150 4750 3150
 Wire Wire Line
-	5050 3250 4050 3250
-Wire Wire Line
-	5050 3350 3600 3350
-Wire Wire Line
-	5050 3450 3900 3450
+	5050 3250 3550 3250
+Wire Wire Line
+	5050 3350 3100 3350
+Wire Wire Line
+	5050 3450 3350 3450
 Wire Wire Line
 	5050 3750 4950 3750
@@
 Text Notes 9250 2050 2    50   ~ 0
 BYPAS\n
-Text GLabel 3400 2850 0    50   Input ~ 0
+Text GLabel 2700 2700 0    50   Input ~ 0
 RX_I
-Text GLabel 3400 2950 0    50   Input ~ 0
+Text GLabel 2700 2800 0    50   Input ~ 0
 RX_Q
 Text GLabel 7150 3350 2    50   Input ~ 0
@@
 L power:+3V3 #PWR02
 U 1 1 5E38F1B7
-P 3900 2650
-F 0 "#PWR02" H 3900 2500 50  0001 C CNN
-F 1 "+3V3" H 3915 2823 50  0000 C CNN
-F 2 "" H 3900 2650 50  0001 C CNN
-F 3 "" H 3900 2650 50  0001 C CNN
-	1    3900 2650
+P 3350 2650
+F 0 "#PWR02" H 3350 2500 50  0001 C CNN
+F 1 "+3V3" H 3365 2823 50  0000 C CNN
+F 2 "" H 3350 2650 50  0001 C CNN
+F 3 "" H 3350 2650 50  0001 C CNN
+	1    3350 2650
 	1    0    0    -1
 $EndComp
@@
 L power:+5V #PWR05
 U 1 1 5E38C061
-P 4050 2650
-F 0 "#PWR05" H 4050 2500 50  0001 C CNN
-F 1 "+5V" H 4065 2823 50  0000 C CNN
-F 2 "" H 4050 2650 50  0001 C CNN
-F 3 "" H 4050 2650 50  0001 C CNN
-	1    4050 2650
+P 3550 2650
+F 0 "#PWR05" H 3550 2500 50  0001 C CNN
+F 1 "+5V" H 3565 2823 50  0000 C CNN
+F 2 "" H 3550 2650 50  0001 C CNN
+F 3 "" H 3550 2650 50  0001 C CNN
+	1    3550 2650
 	1    0    0    -1
 $EndComp
@@
 L power:GND #PWR01
 U 1 1 5E38B1EC
-P 3600 3850
-F 0 "#PWR01" H 3600 3600 50  0001 C CNN
-F 1 "GND" H 3605 3677 50  0000 C CNN
-F 2 "" H 3600 3850 50  0001 C CNN
-F 3 "" H 3600 3850 50  0001 C CNN
-	1    3600 3850
+P 3100 3850
+F 0 "#PWR01" H 3100 3600 50  0001 C CNN
+F 1 "GND" H 3105 3677 50  0000 C CNN
+F 2 "" H 3100 3850 50  0001 C CNN
+F 3 "" H 3100 3850 50  0001 C CNN
+	1    3100 3850
 	1    0    0    -1
 $EndComp
@@
 L Device:R R1
 U 1 1 5E61E083
-P 4500 3150
-F 0 "R1" V 4706 3150 50  0000 C CNN
-F 1 "1K" V 4615 3150 50  0000 C CNN
-F 2 "Resistor_SMD:R_0805_2012Metric" V 4430 3150 50  0001 C CNN
-F 3 "~" H 4500 3150 50  0001 C CNN
-	1    4500 3150
+P 4000 3150
+F 0 "R1" V 4206 3150 50  0000 C CNN
+F 1 "1K" V 4115 3150 50  0000 C CNN
+F 2 "Resistor_SMD:R_0805_2012Metric" V 3930 3150 50  0001 C CNN
+F 3 "~" H 4000 3150 50  0001 C CNN
+	1    4000 3150
 	0    -1   -1   0
 $EndComp
