File: pcb/openxcvr/rx_mixer.sch (KiCad schematic (older format))
At the start: 36 parts, among them U1 SN74CBT3253, U2 LM4562, U3 LM4562, U4 LM4562

Commit message: Candidate design
Parts:
- removed C1: 100nF, Capacitor_SMD:C_0805_2012Metric, symbol Device:C
- removed R2: 10K, Resistor_SMD:R_0805_2012Metric, symbol Device:R
- C20: renamed from C3; value 100nF -> 100n
- C21: renamed from C4; value 100nF -> 100n
- C22: renamed from C5; value 100nF -> 100n
- C23: renamed from C6; value 100nF -> 100n
- C24: renamed from C7; value 1uF -> 1u
- C25: renamed from C8; value 1uF -> 1u
- C26: renamed from C9; value 1uF -> 1u
- C27: renamed from C10; value 1uF -> 1u
- C28: renamed from C11; value 1uF -> 1u
- C29: renamed from C12; value 1uF -> 1u
- R11: renamed from R1; value 82R -> 82
- R16: renamed from R7; value 150R -> 150
- R17: renamed from R8; value 150R -> 150
- U4: renamed from U1; value SN74CBT3253 -> FST5253; symbol Analog_Switch:SN74CBT3253 -> xcvr_components:FST5253
- renumbered C2 to C19, R3 to R12, R4 to R13, R5 to R14, R6 to R15, R9 to R18, R10 to R19, R11 to R20, R12 to R21, R13 to R22, R14 to R23, R15 to R24, R16 to R25, R17 to R26, R18 to R27, R19 to R28, R20 to R29, U3 to U5, U2 to U5, U3 to U6, U2 to U6, U4 to U7
Connections:
- net labels removed: TRANSMIT_RF
- wire segments 134 -> 127

Commit message: Get things working with rev 1 PCB
Parts:
- removed C24, C25, C26, C27: 1u, Capacitor_SMD:C_0805_2012Metric, symbol Device:C
- removed R12: 10K, Resistor_SMD:R_0805_2012Metric, symbol Device:R
- removed R16, R17: 150, Resistor_SMD:R_0805_2012Metric, symbol Device:R
- removed R19, R20, R21, R23, R24, R25, R26, R27, R28, R29: 2K2, Resistor_SMD:R_0805_2012Metric, symbol Device:R
- removed U6, U7: LM4562, Package_SO:SOIC-8_3.9x4.9mm_P1.27mm, symbol Amplifier_Operational:LM4562
- added T1: cx2074NL, openxcvr:bn43-2402-transformer, symbol xcvr_components:cx2074NL
- C20, C21: value 100n -> 22n
- C22, C23: value 100n -> 390p
- R13: value 10K -> 82
- R14, R15: value 10K -> 100
Connections:
- net labels removed: I_NEG, I_POS, Q_NEG, Q_POS
- wire segments 127 -> 71
Other:
- moved on the sheet: C19, C28, C29, R11, R18, R22

Commit message: Add eeprom load store capability
Parts:
- C23: renamed from C22; value 390p -> 1n
- C24: renamed from C23; value 390p -> 1n
- T1: value cx2074NL -> BN43-24023
- renumbered C19 to C20, C20 to C21, C21 to C22, C28 to C25, C29 to C26, R11 to R13, R13 to R14, R14 to R15, R15 to R16, R18 to R17, R22 to R18, U5 to U4, U4 to U5
Other:
- note added: "Primary 4T Unifilar\nSecondary 2T Bifilar\n"
Changed lines of the file:
@@
 $Descr A4 11693 8268
 encoding utf-8
-Sheet 4 6
+Sheet 4 7
 Title "Open XCVR"
 Date "2020-01-26"
@@
 Connection ~ 3100 4800
 Connection ~ 4200 4400
-Connection ~ 4300 4200
+Connection ~ 4300 4100
 Connection ~ 6150 3500
 Connection ~ 6150 5100
@@
 	3600 5100 3600 5350
 Wire Wire Line
-	4000 4200 4300 4200
+	4000 4100 4300 4100
 Wire Wire Line
 	4000 4400 4200 4400
@@
 	4000 4600 4200 4600
 Wire Wire Line
-	4000 4800 4300 4800
+	4000 4900 4300 4900
 Wire Wire Line
 	4200 4400 4600 4400
@@
 	4200 4600 4200 4400
 Wire Wire Line
-	4300 4200 4600 4200
-Wire Wire Line
-	4300 4800 4300 4200
+	4300 4100 4300 4900
+Wire Wire Line
+	4300 4100 4600 4100
 Wire Wire Line
 	4600 3500 6150 3500
 Wire Wire Line
-	4600 4200 4600 3500
+	4600 4100 4600 3500
 Wire Wire Line
 	4600 4400 4600 5100
@@
 Wire Wire Line
 	9300 5200 9600 5200
+Text Notes 2200 3450 2    50   ~ 0
+Primary 4T Unifilar\nSecondary 2T Bifilar\n
 Text GLabel 1200 3800 0    50   BiDi ~ 0
 RF_BPF
@@
 RX_Q
 $Comp
-L power:+2V5 #PWR042
+L power:+2V5 #PWR041
 U 1 1 5E6A7FCA
 P 2350 3900
-F 0 "#PWR042" H 2350 3750 50  0001 C CNN
+F 0 "#PWR041" H 2350 3750 50  0001 C CNN
 F 1 "+2V5" H 2365 4073 50  0000 C CNN
 F 2 "" H 2350 3900 50  0001 C CNN
@@
 $EndComp
 $Comp
-L power:+5V #PWR039
+L power:+5V #PWR042
 U 1 1 5E2E2ABD
 P 3200 1100
-F 0 "#PWR039" H 3200 950 50  0001 C CNN
+F 0 "#PWR042" H 3200 950 50  0001 C CNN
 F 1 "+5V" H 3215 1273 50  0000 C CNN
 F 2 "" H 3200 1100 50  0001 C CNN
@@
 $EndComp
 $Comp
-L power:+5V #PWR045
+L power:+5V #PWR044
 U 1 1 5E41F324
 P 3550 1150
-F 0 "#PWR045" H 3550 1000 50  0001 C CNN
+F 0 "#PWR044" H 3550 1000 50  0001 C CNN
 F 1 "+5V" H 3565 1323 50  0000 C CNN
 F 2 "" H 3550 1150 50  0001 C CNN
@@
 $EndComp
 $Comp
-L power:+5V #PWR037
+L power:+5V #PWR046
 U 1 1 5E3043EB
 P 3600 3800
-F 0 "#PWR037" H 3600 3650 50  0001 C CNN
+F 0 "#PWR046" H 3600 3650 50  0001 C CNN
 F 1 "+5V" H 3615 3973 50  0000 C CNN
 F 2 "" H 3600 3800 50  0001 C CNN
@@
 $EndComp
 $Comp
-L power:+2V5 #PWR047
+L power:+2V5 #PWR050
 U 1 1 5E6C5245
 P 7500 3300
-F 0 "#PWR047" H 7500 3150 50  0001 C CNN
+F 0 "#PWR050" H 7500 3150 50  0001 C CNN
 F 1 "+2V5" H 7515 3473 50  0000 C CNN
 F 2 "" H 7500 3300 50  0001 C CNN
@@
 $EndComp
 $Comp
-L power:GND #PWR041
+L power:GND #PWR040
 U 1 1 5E6A9694
 P 1050 4500
-F 0 "#PWR041" H 1050 4250 50  0001 C CNN
+F 0 "#PWR040" H 1050 4250 50  0001 C CNN
 F 1 "GND" H 1055 4327 50  0000 C CNN
 F 2 "" H 1050 4500 50  0001 C CNN
@@
 $EndComp
 $Comp
-L power:GND #PWR040
+L power:GND #PWR043
 U 1 1 5E2E1D5D
 P 3200 1850
-F 0 "#PWR040" H 3200 1600 50  0001 C CNN
+F 0 "#PWR043" H 3200 1600 50  0001 C CNN
 F 1 "GND" H 3205 1677 50  0000 C CNN
 F 2 "" H 3200 1850 50  0001 C CNN
@@
 $EndComp
 $Comp
-L power:GND #PWR046
+L power:GND #PWR045
 U 1 1 5E418F7E
 P 3550 1700
-F 0 "#PWR046" H 3550 1450 50  0001 C CNN
+F 0 "#PWR045" H 3550 1450 50  0001 C CNN
 F 1 "GND" H 3555 1527 50  0000 C CNN
 F 2 "" H 3550 1700 50  0001 C CNN
@@
 $EndComp
 $Comp
-L power:GND #PWR038
+L power:GND #PWR047
 U 1 1 5E2FDE55
 P 3600 5350
-F 0 "#PWR038" H 3600 5100 50  0001 C CNN
+F 0 "#PWR047" H 3600 5100 50  0001 C CNN
 F 1 "GND" H 3605 5177 50  0000 C CNN
 F 2 "" H 3600 5350 50  0001 C CNN
@@
 $EndComp
 $Comp
-L power:GND #PWR043
+L power:GND #PWR048
 U 1 1 5E73DEF2
 P 6150 4150
-F 0 "#PWR043" H 6150 3900 50  0001 C CNN
+F 0 "#PWR048" H 6150 3900 50  0001 C CNN
 F 1 "GND" H 6155 3977 50  0000 C CNN
 F 2 "" H 6150 4150 50  0001 C CNN
@@
 $EndComp
 $Comp
-L power:GND #PWR044
+L power:GND #PWR049
 U 1 1 5E73A28C
 P 6150 5750
-F 0 "#PWR044" H 6150 5500 50  0001 C CNN
+F 0 "#PWR049" H 6150 5500 50  0001 C CNN
 F 1 "GND" H 6155 5577 50  0000 C CNN
 F 2 "" H 6150 5750 50  0001 C CNN
@@
 $EndComp
 $Comp
-L Device:R R11
+L Device:R R13
 U 1 1 5E2D04D7
 P 2650 3800
-F 0 "R11" V 2856 3800 50  0000 C CNN
+F 0 "R13" V 2856 3800 50  0000 C CNN
 F 1 "82" V 2765 3800 50  0000 C CNN
 F 2 "Resistor_SMD:R_0805_2012Metric" V 2580 3800 50  0001 C CNN
@@
 $EndComp
 $Comp
-L Device:R R13
+L Device:R R14
 U 1 1 5E7EE68A
 P 2650 4200
-F 0 "R13" V 2856 4200 50  0000 C CNN
+F 0 "R14" V 2856 4200 50  0000 C CNN
 F 1 "82" V 2765 4200 50  0000 C CNN
 F 2 "Resistor_SMD:R_0805_2012Metric" V 2580 4200 50  0001 C CNN
@@
 $EndComp
 $Comp
-L Device:R R14
+L Device:R R15
 U 1 1 5E6B255C
 P 7000 3500
-F 0 "R14" H 6930 3455 50  0000 R CNN
+F 0 "R15" H 6930 3455 50  0000 R CNN
 F 1 "100" H 6930 3545 50  0000 R CNN
 F 2 "Resistor_SMD:R_0805_2012Metric" V 6930 3500 50  0001 C CNN
@@
 $EndComp
 $Comp
-L Device:R R15
+L Device:R R16
 U 1 1 5E70FAD3
 P 7000 5100
-F 0 "R15" H 6930 5055 50  0000 R CNN
+F 0 "R16" H 6930 5055 50  0000 R CNN
 F 1 "100" H 6930 5145 50  0000 R CNN
 F 2 "Resistor_SMD:R_0805_2012Metric" V 6930 5100 50  0001 C CNN
@@
 $EndComp
 $Comp
-L Device:R R18
+L Device:R R17
 U 1 1 5E2682B3
 P 8250 3200
-F 0 "R18" V 8456 3200 50  0000 C CNN
+F 0 "R17" V 8456 3200 50  0000 C CNN
 F 1 "2K2" V 8365 3200 50  0000 C CNN
 F 2 "Resistor_SMD:R_0805_2012Metric" V 8180 3200 50  0001 C CNN
@@
 $EndComp
 $Comp
-L Device:R R22
+L Device:R R18
 U 1 1 5E268EC4
 P 8250 4800
-F 0 "R22" V 8456 4800 50  0000 C CNN
+F 0 "R18" V 8456 4800 50  0000 C CNN
 F 1 "2K2" V 8365 4800 50  0000 C CNN
 F 2 "Resistor_SMD:R_0805_2012Metric" V 8180 4800 50  0001 C CNN
@@
 $EndComp
 $Comp
-L Amplifier_Operational:LM4562 U5
+L Amplifier_Operational:LM4562 U4
 U 3 1 5E262A9E
 P 3300 1450
-F 0 "U5" H 3200 2100 50  0000 C CNN
+F 0 "U4" H 3200 2100 50  0000 C CNN
 F 1 "LM4562" H 3200 1450 50  0000 C CNN
 F 2 "Package_SO:SOIC-8_3.9x4.9mm_P1.27mm" H 3300 1450 50  0001 C CNN
@@
 $EndComp
 $Comp
-L Device:C C19
+L Device:C C20
 U 1 1 5E418F5E
 P 3550 1450
-F 0 "C19" H 3665 1495 50  0000 L CNN
+F 0 "C20" H 3665 1495 50  0000 L CNN
 F 1 "100n" H 3665 1405 50  0000 L CNN
 F 2 "Capacitor_SMD:C_0805_2012Metric" H 3588 1300 50  0001 C CNN
@@
 $EndComp
 $Comp
-L Device:C C20
+L Device:C C21
 U 1 1 5E72F21F
 P 6150 3850
-F 0 "C20" V 6401 3850 50  0000 C CNN
+F 0 "C21" V 6401 3850 50  0000 C CNN
 F 1 "22n" V 6310 3850 50  0000 C CNN
 F 2 "Capacitor_SMD:C_0805_2012Metric" H 6188 3700 50  0001 C CNN
@@
 $EndComp
 $Comp
-L Device:C C21
+L Device:C C22
 U 1 1 5E7357AF
 P 6150 5450
-F 0 "C21" V 6401 5450 50  0000 C CNN
+F 0 "C22" V 6401 5450 50  0000 C CNN
 F 1 "22n" V 6310 5450 50  0000 C CNN
 F 2 "Capacitor_SMD:C_0805_2012Metric" H 6188 5300 50  0001 C CNN
@@
 $EndComp
 $Comp
-L Device:C C22
+L Device:C C23
 U 1 1 5E72984C
 P 8250 2750
-F 0 "C22" V 8501 2750 50  0000 C CNN
-F 1 "390p" V 8410 2750 50  0000 C CNN
+F 0 "C23" V 8501 2750 50  0000 C CNN
+F 1 "1n" V 8410 2750 50  0000 C CNN
 F 2 "Capacitor_SMD:C_0805_2012Metric" H 8288 2600 50  0001 C CNN
 F 3 "~" H 8250 2750 50  0001 C CNN
@@
 $EndComp
 $Comp
-L Device:C C23
+L Device:C C24
 U 1 1 5E729FA5
 P 8250 4400
-F 0 "C23" V 8501 4400 50  0000 C CNN
-F 1 "390p" V 8410 4400 50  0000 C CNN
+F 0 "C24" V 8501 4400 50  0000 C CNN
+F 1 "1n" V 8410 4400 50  0000 C CNN
 F 2 "Capacitor_SMD:C_0805_2012Metric" H 8288 4250 50  0001 C CNN
 F 3 "~" H 8250 4400 50  0001 C CNN
@@
 $EndComp
 $Comp
-L Device:C C28
+L Device:C C25
 U 1 1 5E26B729
 P 9150 3600
-F 0 "C28" V 9401 3600 50  0000 C CNN
+F 0 "C25" V 9401 3600 50  0000 C CNN
 F 1 "1u" V 9310 3600 50  0000 C CNN
 F 2 "Capacitor_SMD:C_0805_2012Metric" H 9188 3450 50  0001 C CNN
@@
 $EndComp
 $Comp
-L Device:C C29
+L Device:C C26
 U 1 1 5E38AC32
 P 9150 5200
-F 0 "C29" V 9401 5200 50  0000 C CNN
+F 0 "C26" V 9401 5200 50  0000 C CNN
 F 1 "1u" V 9310 5200 50  0000 C CNN
 F 2 "Capacitor_SMD:C_0805_2012Metric" H 9188 5050 50  0001 C CNN
@@
 $EndComp
 $Comp
-L Amplifier_Operational:LM4562 U5
+L Amplifier_Operational:LM4562 U4
 U 2 1 5E26166E
 P 8250 3600
-F 0 "U5" H 8250 3966 50  0000 C CNN
+F 0 "U4" H 8250 3966 50  0000 C CNN
 F 1 "LM4562" H 8250 3875 50  0000 C CNN
 F 2 "Package_SO:SOIC-8_3.9x4.9mm_P1.27mm" H 8250 3600 50  0001 C CNN
@@
 $EndComp
 $Comp
-L Amplifier_Operational:LM4562 U5
+L Amplifier_Operational:LM4562 U4
 U 1 1 5E262689
 P 8250 5200
-F 0 "U5" H 8250 5400 50  0000 C CNN
+F 0 "U4" H 8250 5400 50  0000 C CNN
 F 1 "LM4562" H 8250 5500 50  0000 C CNN
 F 2 "Package_SO:SOIC-8_3.9x4.9mm_P1.27mm" H 8250 5200 50  0001 C CNN
@@
 P 1800 4000
 F 0 "T1" H 1800 4379 50  0000 C CNN
-F 1 "cx2074NL" H 1800 4288 50  0000 C CNN
+F 1 "BN43-24023" H 1800 4288 50  0000 C CNN
 F 2 "openxcvr:bn43-2402-transformer" H 1800 4000 50  0001 C CNN
 F 3 "https://datasheet.octopart.com/CX2074NL-Pulse-datasheet-123678.pdf" H 1800 4000 50  0001 C CNN
@@
 $EndComp
 $Comp
-L xcvr_components:FST5253 U4
+L xcvr_components:FST5253 U5
 U 1 1 5E2AF6E6
 P 3600 4500
-F 0 "U4" H 4000 5200 50  0000 C CNN
+F 0 "U5" H 4000 5200 50  0000 C CNN
 F 1 "FST5253" H 4000 5100 50  0000 C CNN
 F 2 "Package_SO:SOIC-16_3.9x9.9mm_P1.27mm" H 3600 4500 50  0001 C CNN

Commit message: update rev0.2 PCB
Parts:
- added C51: 100n, Capacitor_SMD:C_0805_2012Metric, symbol Device:C
- added J8: Conn_01x03_Male, Connector_PinHeader_2.54mm:PinHeader_1x03_P2.54mm_Vertical, symbol Connector:Conn_01x03_Male
- T1: value BN43-24023 -> BN43-2402; symbol xcvr_components:cx2074NL -> RADIO-rescue:cx2074NL-xcvr_components
- U5: symbol xcvr_components:FST5253 -> RADIO-rescue:FST5253-xcvr_components
Connections:
- wire segments 71 -> 81
Changed lines of the file:
@@
 Connection ~ 8750 4800
 Connection ~ 8750 5200
+Connection ~ 9450 3600
+Connection ~ 9450 5200
 Wire Wire Line
 	1050 4200 1400 4200
@@
 	3600 5100 3600 5350
 Wire Wire Line
+	4000 1150 4000 1300
+Wire Wire Line
+	4000 1600 4000 1700
+Wire Wire Line
 	4000 4100 4300 4100
 Wire Wire Line
@@
 	8750 5200 9000 5200
 Wire Wire Line
-	9300 3600 9600 3600
-Wire Wire Line
-	9300 5200 9600 5200
+	9100 4200 9450 4200
+Wire Wire Line
+	9100 4300 9800 4300
+Wire Wire Line
+	9100 4400 9450 4400
+Wire Wire Line
+	9300 3600 9450 3600
+Wire Wire Line
+	9300 5200 9450 5200
+Wire Wire Line
+	9450 3600 9600 3600
+Wire Wire Line
+	9450 4200 9450 3600
+Wire Wire Line
+	9450 4400 9450 5200
+Wire Wire Line
+	9450 5200 9600 5200
+Wire Wire Line
+	9800 4300 9800 4600
 Text Notes 2200 3450 2    50   ~ 0
 Primary 4T Unifilar\nSecondary 2T Bifilar\n
@@
 $EndComp
 $Comp
+L power:+5V #PWR0102
+U 1 1 5ECD0B83
+P 4000 1150
+F 0 "#PWR0102" H 4000 1000 50  0001 C CNN
+F 1 "+5V" H 4015 1323 50  0000 C CNN
+F 2 "" H 4000 1150 50  0001 C CNN
+F 3 "" H 4000 1150 50  0001 C CNN
+	1    4000 1150
+	1    0    0    -1
+$EndComp
+$Comp
 L power:+2V5 #PWR050
 U 1 1 5E6C5245
@@
 $EndComp
 $Comp
+L power:GND #PWR0103
+U 1 1 5ECD0B93
+P 4000 1700
+F 0 "#PWR0103" H 4000 1450 50  0001 C CNN
+F 1 "GND" H 4005 1527 50  0000 C CNN
+F 2 "" H 4000 1700 50  0001 C CNN
+F 3 "" H 4000 1700 50  0001 C CNN
+	1    4000 1700
+	1    0    0    -1
+$EndComp
+$Comp
 L power:GND #PWR048
 U 1 1 5E73DEF2
@@
 F 3 "" H 6150 5750 50  0001 C CNN
 	1    6150 5750
+	1    0    0    -1
+$EndComp
+$Comp
+L power:GND #PWR0105
+U 1 1 5EDC0D6C
+P 9800 4600
+F 0 "#PWR0105" H 9800 4350 50  0001 C CNN
+F 1 "GND" H 9805 4427 50  0000 C CNN
+F 2 "" H 9800 4600 50  0001 C CNN
+F 3 "" H 9800 4600 50  0001 C CNN
+	1    9800 4600
 	1    0    0    -1
 $EndComp
@@
 $EndComp
 $Comp
+L Device:C C51
+U 1 1 5ECD0BA5
+P 4000 1450
+F 0 "C51" H 4115 1495 50  0000 L CNN
+F 1 "100n" H 4115 1405 50  0000 L CNN
+F 2 "Capacitor_SMD:C_0805_2012Metric" H 4038 1300 50  0001 C CNN
+F 3 "~" H 4000 1450 50  0001 C CNN
+	1    4000 1450
+	1    0    0    -1
+$EndComp
+$Comp
 L Device:C C21
 U 1 1 5E72F21F
@@
 $EndComp
 $Comp
+L Connector:Conn_01x03_Male J8
+U 1 1 5EDBE7DA
+P 8900 4300
+F 0 "J8" H 9008 4579 50  0000 C CNN
+F 1 "Conn_01x03_Male" H 9008 4488 50  0000 C CNN
+F 2 "Connector_PinHeader_2.54mm:PinHeader_1x03_P2.54mm_Vertical" H 8900 4300 50  0001 C CNN
+F 3 "~" H 8900 4300 50  0001 C CNN
+	1    8900 4300
+	1    0    0    -1
+$EndComp
+$Comp
 L Amplifier_Operational:LM4562 U4
 U 2 1 5E26166E
@@
 $EndComp
 $Comp
-L xcvr_components:cx2074NL T1
+L RADIO-rescue:cx2074NL-xcvr_components T1
 U 1 1 5E6894D6
 P 1800 4000
 F 0 "T1" H 1800 4379 50  0000 C CNN
-F 1 "BN43-24023" H 1800 4288 50  0000 C CNN
+F 1 "BN43-2402" H 1800 4288 50  0000 C CNN
 F 2 "openxcvr:bn43-2402-transformer" H 1800 4000 50  0001 C CNN
 F 3 "https://datasheet.octopart.com/CX2074NL-Pulse-datasheet-123678.pdf" H 1800 4000 50  0001 C CNN
@@
 $EndComp
 $Comp
-L xcvr_components:FST5253 U5
+L RADIO-rescue:FST5253-xcvr_components U5
 U 1 1 5E2AF6E6
 P 3600 4500
+AR Path="/5E2AF6E6" Ref="U5"  Part="1"
+AR Path="/5E35BCF5/5E2AF6E6" Ref="U5"  Part="1"
 F 0 "U5" H 4000 5200 50  0000 C CNN
 F 1 "FST5253" H 4000 5100 50  0000 C CNN

Commit message: Review and update schematic
Parts:
- U5: value FST5253 -> FST3253
Connections:
- no-connect marks 0 -> 4
Changed lines of the file:
@@
 $EndDescr
 Connection ~ 3100 4800
-Connection ~ 4200 4400
-Connection ~ 4300 4100
+Connection ~ 4200 4100
+Connection ~ 4250 4200
 Connection ~ 6150 3500
 Connection ~ 6150 5100
@@
 Connection ~ 9450 3600
 Connection ~ 9450 5200
+NoConn ~ 4000 4300
+NoConn ~ 4000 4400
+NoConn ~ 4000 4600
+NoConn ~ 4000 4700
 Wire Wire Line
 	1050 4200 1400 4200
@@
 	4000 1600 4000 1700
 Wire Wire Line
-	4000 4100 4300 4100
-Wire Wire Line
-	4000 4400 4200 4400
-Wire Wire Line
-	4000 4600 4200 4600
-Wire Wire Line
-	4000 4900 4300 4900
-Wire Wire Line
-	4200 4400 4600 4400
-Wire Wire Line
-	4200 4600 4200 4400
-Wire Wire Line
-	4300 4100 4300 4900
-Wire Wire Line
-	4300 4100 4600 4100
+	4000 4100 4200 4100
+Wire Wire Line
+	4000 4200 4250 4200
+Wire Wire Line
+	4000 4800 4250 4800
+Wire Wire Line
+	4000 4900 4200 4900
+Wire Wire Line
+	4200 4100 4600 4100
+Wire Wire Line
+	4200 4900 4200 4100
+Wire Wire Line
+	4250 4200 4600 4200
+Wire Wire Line
+	4250 4800 4250 4200
 Wire Wire Line
 	4600 3500 6150 3500
@@
 	4600 4100 4600 3500
 Wire Wire Line
-	4600 4400 4600 5100
+	4600 4200 4600 5100
 Wire Wire Line
 	4600 5100 6150 5100
@@
 AR Path="/5E35BCF5/5E2AF6E6" Ref="U5"  Part="1"
 F 0 "U5" H 4000 5200 50  0000 C CNN
-F 1 "FST5253" H 4000 5100 50  0000 C CNN
+F 1 "FST3253" H 4000 5100 50  0000 C CNN
 F 2 "Package_SO:SOIC-16_3.9x9.9mm_P1.27mm" H 3600 4500 50  0001 C CNN
 F 3 "http://www.ti.com/lit/gpn/sn74cbt3253" H 3600 4500 50  0001 C CNN

Commit message: Review schematic and PCB layout
Parts:
- J8: value Conn_01x03_Male -> IQ TEST
Connections:
- wire segments 81 -> 83
Other:
- moved on the sheet: R13
Changed lines of the file:
@@
 $Descr A4 11693 8268
 encoding utf-8
-Sheet 4 7
+Sheet 3 7
 Title "Open XCVR"
-Date "2020-01-26"
-Rev "0.1"
+Date "2020-06-14"
+Rev "0.2"
 Comp "Jon Dawson"
 Comment1 ""
@@
 	1200 3800 1400 3800
 Wire Wire Line
-	2200 3800 2500 3800
+	2200 3800 2250 3800
 Wire Wire Line
 	2200 4000 2350 4000
@@
 	2200 4200 2500 4200
 Wire Wire Line
+	2250 3550 2500 3550
+Wire Wire Line
+	2250 3800 2250 3550
+Wire Wire Line
 	2350 4000 2350 3900
 Wire Wire Line
@@
 	2350 4800 3100 4800
 Wire Wire Line
-	2800 3800 3000 3800
+	2800 3550 3000 3550
 Wire Wire Line
 	2800 4200 3200 4200
 Wire Wire Line
-	3000 3800 3000 4100
+	3000 3550 3000 4100
 Wire Wire Line
 	3000 4100 3200 4100
@@
 L Device:R R13
 U 1 1 5E2D04D7
-P 2650 3800
-F 0 "R13" V 2856 3800 50  0000 C CNN
-F 1 "82" V 2765 3800 50  0000 C CNN
-F 2 "Resistor_SMD:R_0805_2012Metric" V 2580 3800 50  0001 C CNN
-F 3 "~" H 2650 3800 50  0001 C CNN
-	1    2650 3800
+P 2650 3550
+F 0 "R13" V 2856 3550 50  0000 C CNN
+F 1 "82" V 2765 3550 50  0000 C CNN
+F 2 "Resistor_SMD:R_0805_2012Metric" V 2580 3550 50  0001 C CNN
+F 3 "~" H 2650 3550 50  0001 C CNN
+	1    2650 3550
 	0    -1   -1   0
 $EndComp
@@
 U 1 1 5EDBE7DA
 P 8900 4300
-F 0 "J8" H 9008 4579 50  0000 C CNN
-F 1 "Conn_01x03_Male" H 9008 4488 50  0000 C CNN
+F 0 "J8" H 9000 4600 50  0000 C CNN
+F 1 "IQ TEST" H 9050 4500 50  0000 C CNN
 F 2 "Connector_PinHeader_2.54mm:PinHeader_1x03_P2.54mm_Vertical" H 8900 4300 50  0001 C CNN
 F 3 "~" H 8900 4300 50  0001 C CNN
