File: pcb/openxcvr/tx_pa.sch (KiCad schematic (older format))
At the start: 25 parts, among them Q4 BS170, Q5 BS170, Q6 BS170, U4 MCP1406, U5 DMC3056LSS, U6 74AC00

Commit message: Review and update schematic
Parts:
- added R19, R21: 10k, Resistor_SMD:R_0805_2012Metric, symbol Device:R
- C27: value C -> 100n
Connections:
- wire segments 121 -> 127
Other:
- moved on the sheet: C21, C22, C23, C24, C25, C26, C27, C28, D7, D8, L13, L14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

Commit message: Review schematic and PCB layout
Parts:
- L15: value L -> 44 u
Other:
- note added: "Envelope (audio) switching amplifier"
- note added: "FT 50-43 10 Turns"
- note added: "RF switching amplifier"
- moved on the sheet: C27, R14, R15, R19, U4
Changed lines of the file:
@@
 encoding utf-8
 Sheet 3 4
-Title ""
-Date ""
-Rev ""
-Comp ""
+Title "Open XCVR"
+Date "2020-06-14"
+Rev "0.2"
+Comp "Jon Dawson"
 Comment1 ""
 Comment2 ""
@@
 Comment9 ""
 $EndDescr
-Connection ~ 2250 1450
-Connection ~ 3050 1000
-Connection ~ 3050 2100
-Connection ~ 3550 1550
-Connection ~ 3600 1650
+Connection ~ 1600 1400
+Connection ~ 2400 950
+Connection ~ 2400 2050
+Connection ~ 2900 1500
+Connection ~ 3200 1650
+Connection ~ 3650 1650
 Connection ~ 3900 1350
 Connection ~ 3900 1450
 Connection ~ 3950 4750
-Connection ~ 4050 1650
 Connection ~ 4250 3300
 Connection ~ 4250 3650
@@
 Connection ~ 10000 5800
 Wire Wire Line
-	1950 1450 2250 1450
-Wire Wire Line
-	2250 1450 2250 2150
-Wire Wire Line
-	2250 1450 2650 1450
-Wire Wire Line
-	2250 2450 2250 2750
-Wire Wire Line
-	2550 1000 3050 1000
-Wire Wire Line
-	2550 1350 2550 1000
-Wire Wire Line
-	2550 1650 2650 1650
-Wire Wire Line
-	2550 2100 2550 1650
-Wire Wire Line
-	2650 1350 2550 1350
-Wire Wire Line
-	3050 900  3050 1000
-Wire Wire Line
-	3050 1000 3550 1000
-Wire Wire Line
-	3050 2100 2550 2100
-Wire Wire Line
-	3050 2100 3050 2200
+	1300 1400 1600 1400
+Wire Wire Line
+	1600 1400 1600 2100
+Wire Wire Line
+	1600 1400 2000 1400
+Wire Wire Line
+	1600 2400 1600 2700
+Wire Wire Line
+	1900 950  2400 950
+Wire Wire Line
+	1900 1300 1900 950
+Wire Wire Line
+	1900 1600 2000 1600
+Wire Wire Line
+	1900 2050 1900 1600
+Wire Wire Line
+	2000 1300 1900 1300
+Wire Wire Line
+	2400 850  2400 950
+Wire Wire Line
+	2400 950  2900 950
+Wire Wire Line
+	2400 2050 1900 2050
+Wire Wire Line
+	2400 2050 2400 2150
+Wire Wire Line
+	2800 1400 2900 1400
+Wire Wire Line
+	2800 1500 2900 1500
+Wire Wire Line
+	2800 1600 2900 1600
+Wire Wire Line
+	2900 950  2900 1300
+Wire Wire Line
+	2900 1300 2800 1300
+Wire Wire Line
+	2900 1500 2900 1400
+Wire Wire Line
+	2900 1500 3200 1500
+Wire Wire Line
+	2900 1600 2900 2050
+Wire Wire Line
+	2900 2050 2400 2050
+Wire Wire Line
+	3200 1500 3200 1650
+Wire Wire Line
+	3200 1650 3300 1650
+Wire Wire Line
+	3200 1750 3200 1650
 Wire Wire Line
 	3200 4750 3950 4750
@@
 	3200 4950 4400 4950
 Wire Wire Line
-	3450 1450 3550 1450
-Wire Wire Line
-	3450 1550 3550 1550
-Wire Wire Line
-	3450 1650 3550 1650
-Wire Wire Line
-	3550 1000 3550 1350
-Wire Wire Line
-	3550 1350 3450 1350
-Wire Wire Line
-	3550 1550 3550 1450
-Wire Wire Line
-	3550 1650 3550 2100
-Wire Wire Line
-	3550 2100 3050 2100
-Wire Wire Line
-	3600 1550 3550 1550
-Wire Wire Line
-	3600 1650 3600 1550
-Wire Wire Line
-	3600 1650 3700 1650
-Wire Wire Line
-	3600 1750 3600 1650
-Wire Wire Line
-	3700 1750 3600 1750
+	3300 1750 3200 1750
+Wire Wire Line
+	3600 1650 3650 1650
+Wire Wire Line
+	3600 1750 3650 1750
+Wire Wire Line
+	3650 1650 4100 1650
+Wire Wire Line
+	3650 1750 3650 1650
 Wire Wire Line
 	3900 950  3900 1350
@@
 	3950 5500 3950 5800
 Wire Wire Line
-	4000 1650 4050 1650
-Wire Wire Line
-	4000 1750 4050 1750
-Wire Wire Line
-	4050 1650 4100 1650
-Wire Wire Line
-	4050 1750 4050 1650
-Wire Wire Line
 	4100 1550 3900 1550
 Wire Wire Line
@@
 	8350 3950 8350 4550
 Wire Wire Line
+	9450 4700 10000 4700
+Wire Wire Line
+	9450 5100 9450 4700
+Wire Wire Line
+	9450 5400 9450 5800
+Wire Wire Line
+	9450 5800 10000 5800
+Wire Wire Line
 	9550 2800 9650 2800
 Wire Wire Line
-	9550 4700 10000 4700
-Wire Wire Line
-	9550 5100 9550 4700
-Wire Wire Line
-	9550 5400 9550 5800
-Wire Wire Line
-	9550 5800 10000 5800
-Wire Wire Line
 	10000 4650 10000 4700
 Wire Wire Line
@@
 Wire Wire Line
 	10000 5800 10000 5850
-Text GLabel 1950 1450 0    50   Input ~ 0
+Wire Notes Line
+	1300 550  1300 3550
+Wire Notes Line
+	1300 550  6900 550
+Wire Notes Line
+	1300 3550 3900 3550
+Wire Notes Line
+	2250 3600 2250 6200
+Wire Notes Line
+	2250 3600 3950 3600
+Wire Notes Line
+	2250 6200 8700 6200
+Wire Notes Line
+	3900 2550 6150 2550
+Wire Notes Line
+	3900 3550 3900 2550
+Wire Notes Line
+	3950 2600 3950 3600
+Wire Notes Line
+	6150 1950 6900 1950
+Wire Notes Line
+	6150 2550 6150 1950
+Wire Notes Line
+	6200 2000 6200 2600
+Wire Notes Line
+	6200 2600 3950 2600
+Wire Notes Line
+	6900 1950 6900 550
+Wire Notes Line
+	8700 3150 10050 3150
+Wire Notes Line
+	8700 6200 8700 3150
+Wire Notes Line
+	10050 2000 6200 2000
+Wire Notes Line
+	10050 3150 10050 2000
+Text Notes 3600 2750 2    50   ~ 0
+Envelope (audio) switching amplifier
+Text Notes 7600 2450 2    50   ~ 0
+FT 50-43 10 Turns
+Text Notes 8050 5550 2    50   ~ 0
+RF switching amplifier
+Text GLabel 1300 1400 0    50   Input ~ 0
 RF_ENVELOPE
 Text GLabel 3200 4750 0    50   Input ~ 0
@@
 L power:+12V #PWR037
 U 1 1 5EE4DF0B
-P 3050 900
-F 0 "#PWR037" H 3050 750 50  0001 C CNN
-F 1 "+12V" H 3065 1073 50  0000 C CNN
-F 2 "" H 3050 900 50  0001 C CNN
-F 3 "" H 3050 900 50  0001 C CNN
-	1    3050 900
+P 2400 850
+F 0 "#PWR037" H 2400 700 50  0001 C CNN
+F 1 "+12V" H 2415 1023 50  0000 C CNN
+F 2 "" H 2400 850 50  0001 C CNN
+F 3 "" H 2400 850 50  0001 C CNN
+	1    2400 850
 	1    0    0    -1
 $EndComp
@@
 L power:GND #PWR0101
 U 1 1 5EF0B36C
-P 2250 2750
-F 0 "#PWR0101" H 2250 2500 50  0001 C CNN
-F 1 "GND" H 2255 2577 50  0000 C CNN
-F 2 "" H 2250 2750 50  0001 C CNN
-F 3 "" H 2250 2750 50  0001 C CNN
-	1    2250 2750
+P 1600 2700
+F 0 "#PWR0101" H 1600 2450 50  0001 C CNN
+F 1 "GND" H 1605 2527 50  0000 C CNN
+F 2 "" H 1600 2700 50  0001 C CNN
+F 3 "" H 1600 2700 50  0001 C CNN
+	1    1600 2700
 	1    0    0    -1
 $EndComp
@@
 L power:GND #PWR038
 U 1 1 5EE4D545
-P 3050 2200
-F 0 "#PWR038" H 3050 1950 50  0001 C CNN
-F 1 "GND" H 3055 2027 50  0000 C CNN
-F 2 "" H 3050 2200 50  0001 C CNN
-F 3 "" H 3050 2200 50  0001 C CNN
-	1    3050 2200
+P 2400 2150
+F 0 "#PWR038" H 2400 1900 50  0001 C CNN
+F 1 "GND" H 2405 1977 50  0000 C CNN
+F 2 "" H 2400 2150 50  0001 C CNN
+F 3 "" H 2400 2150 50  0001 C CNN
+	1    2400 2150
 	1    0    0    -1
 $EndComp
@@
 P 6500 2400
 F 0 "L15" H 6553 2445 50  0000 L CNN
-F 1 "L" H 6553 2355 50  0000 L CNN
+F 1 "44 u" H 6553 2355 50  0000 L CNN
 F 2 "openxcvr:FT50-43 INDUCTOR" H 6500 2400 50  0001 C CNN
 F 3 "~" H 6500 2400 50  0001 C CNN
@@
 L Device:R R19
 U 1 1 5EF0B35C
-P 2250 2300
-F 0 "R19" H 2320 2345 50  0000 L CNN
-F 1 "10k" H 2320 2255 50  0000 L CNN
-F 2 "Resistor_SMD:R_0805_2012Metric" V 2180 2300 50  0001 C CNN
-F 3 "~" H 2250 2300 50  0001 C CNN
-	1    2250 2300
+P 1600 2250
+F 0 "R19" H 1670 2295 50  0000 L CNN
+F 1 "10k" H 1670 2205 50  0000 L CNN
+F 2 "Resistor_SMD:R_0805_2012Metric" V 1530 2250 50  0001 C CNN
+F 3 "~" H 1600 2250 50  0001 C CNN
+	1    1600 2250
 	1    0    0    -1
 $EndComp
@@
 L Device:R R14
 U 1 1 5EE22A3C
-P 3850 1650
-F 0 "R14" V 3950 1700 50  0000 C CNN
-F 1 "10" V 3950 1800 50  0000 C CNN
-F 2 "Resistor_SMD:R_0805_2012Metric" V 3780 1650 50  0001 C CNN
-F 3 "~" H 3850 1650 50  0001 C CNN
-	1    3850 1650
+P 3450 1650
+F 0 "R14" V 3550 1650 50  0000 C CNN
+F 1 "10" V 3650 1650 50  0000 C CNN
+F 2 "Resistor_SMD:R_0805_2012Metric" V 3380 1650 50  0001 C CNN
+F 3 "~" H 3450 1650 50  0001 C CNN
+	1    3450 1650
 	0    -1   -1   0
 $EndComp
@@
 L Device:R R15
 U 1 1 5EE232F1
-P 3850 1750
-F 0 "R15" V 3750 1650 50  0000 C CNN
-F 1 "10" V 3750 1750 50  0000 C CNN
-F 2 "Resistor_SMD:R_0805_2012Metric" V 3780 1750 50  0001 C CNN
-F 3 "~" H 3850 1750 50  0001 C CNN
-	1    3850 1750
+P 3450 1750
+F 0 "R15" V 3250 1750 50  0000 C CNN
+F 1 "10" V 3350 1750 50  0000 C CNN
+F 2 "Resistor_SMD:R_0805_2012Metric" V 3380 1750 50  0001 C CNN
+F 3 "~" H 3450 1750 50  0001 C CNN
+	1    3450 1750
 	0    -1   -1   0
 $EndComp
@@
 L Device:C C27
 U 1 1 5EEF3AB1
-P 9550 5250
-F 0 "C27" H 9665 5295 50  0000 L CNN
-F 1 "100n" H 9665 5205 50  0000 L CNN
-F 2 "Capacitor_SMD:C_0805_2012Metric" H 9588 5100 50  0001 C CNN
-F 3 "~" H 9550 5250 50  0001 C CNN
-	1    9550 5250
+P 9450 5250
+F 0 "C27" H 9565 5295 50  0000 L CNN
+F 1 "100n" H 9565 5205 50  0000 L CNN
+F 2 "Capacitor_SMD:C_0805_2012Metric" H 9488 5100 50  0001 C CNN
+F 3 "~" H 9450 5250 50  0001 C CNN
+	1    9450 5250
 	1    0    0    -1
 $EndComp
@@
 L xcvr_components:MCP1406 U4
 U 1 1 5EE20EC8
-P 3050 1200
-F 0 "U4" H 3050 1314 50  0000 C CNN
-F 1 "MCP1406" H 3050 1223 50  0000 C CNN
-F 2 "Package_SO:SOIC-8_3.9x4.9mm_P1.27mm" H 3050 1200 50  0001 C CNN
-F 3 "http://ww1.microchip.com/downloads/en/DeviceDoc/20002019C.pdf" H 3050 1200 50  0001 C CNN
-	1    3050 1200
-	1    0    0    -1
-$EndComp
+P 2400 1150
+F 0 "U4" H 2400 1264 50  0000 C CNN
+F 1 "MCP1406" H 2400 1173 50  0000 C CNN
+F 2 "Package_SO:SOIC-8_3.9x4.9mm_P1.27mm" H 2400 1150 50  0001 C CNN
+F 3 "http://ww1.microchip.com/downloads/en/DeviceDoc/20002019C.pdf" H 2400 1150 50  0001 C CNN
+	1    2400 1150
+	1    0    0    -1
+$EndComp
