File: pcb/openxcvr/user_interface.sch (KiCad schematic (older format))
At the start: 22 parts, among them J7 PTT, SW1 SW_Push, SW2 SW_Push, SW3 SW_Push, SW4 SW_Push, SW5 Rotary_Encoder_Switch

Commit message: Review schematic and PCB layout
Other:
- note added: "Contrast"
Changed lines of the file:
@@
 encoding utf-8
 Sheet 7 7
-Title ""
-Date ""
-Rev ""
-Comp ""
+Title "Open XCVR"
+Date "2020-06-14"
+Rev "0.2"
+Comp "Jon Dawson"
 Comment1 ""
 Comment2 ""
@@
 Wire Wire Line
 	8700 2150 8700 2050
+Text Notes 4400 1750 2    50   ~ 0
+Contrast
 Text GLabel 1350 1700 0    50   Input ~ 0
 LCD_E
