File: pcb/openxcvr/audio.sch (KiCad schematic (older format))
At the start: 24 parts, among them U5 LM386, U6 MCP6002-xSN

Commit message: Candidate design
Parts:
- C10: renamed from C14; value 47nF -> 47n
- C14: renamed from C18; value 47nF -> 47n
- C15: renamed from C19; value 100uF -> 100u
- renumbered C15 to C11, C16 to C12, C17 to C13, C20 to C16, C21 to C17, C22 to C18, C13 to C9, R21 to R1, R30 to R10, R22 to R2, R23 to R3, R24 to R4, R25 to R5, R26 to R6, R27 to R7, R28 to R8, R29 to R9, U5 to U2, U6 to U3

Commit message: Get things working with rev 1 PCB
Parts:
- added C24: 100n, Capacitor_SMD:C_0805_2012Metric, symbol Device:C
- RV1, RV2: footprint Potentiometer_THT:Potentiometer_Piher_PT-6-V_Vertical -> Potentiometer_THT:Potentiometer_Piher_PT-6-H_Horizontal
Connections:
- wire segments 85 -> 86
Changed lines of the file:
@@
 NoConn ~ 4550 2300
+Wire Wire Line
+	1750 1200 1900 1200
 Wire Wire Line
 	2150 5050 2450 5050
@@
 Text Notes 7250 3400 2    50   ~ 0
 5v Power Rail Splitter
+Text GLabel 1750 1200 0    50   Input ~ 0
+SPEAKER
 Text GLabel 2150 5050 0    50   Input ~ 0
 MIC_HDR
-Text GLabel 2200 1200 0    50   Input ~ 0
-SPEAKER
 Text GLabel 5625 5300 2    50   Output ~ 0
 MIC
@@
 $EndComp
 $Comp
+L Device:C C24
+U 1 1 5E7745A5
+P 2050 1200
+F 0 "C24" H 2165 1245 50  0000 L CNN
+F 1 "100n" H 2165 1155 50  0000 L CNN
+F 2 "Capacitor_SMD:C_0805_2012Metric" H 2088 1050 50  0001 C CNN
+F 3 "~" H 2050 1200 50  0001 C CNN
+	1    2050 1200
+	0    -1   -1   0
+$EndComp
+$Comp
 L Device:C C9
 U 1 1 5E2F6946
@@
 F 0 "RV1" H 3305 5445 50  0000 R CNN
 F 1 "10K" H 3305 5355 50  0000 R CNN
-F 2 "Potentiometer_THT:Potentiometer_Piher_PT-6-V_Vertical" H 3375 5400 50  0001 C CNN
+F 2 "Potentiometer_THT:Potentiometer_Piher_PT-6-H_Horizontal" H 3375 5400 50  0001 C CNN
 F 3 "~" H 3375 5400 50  0001 C CNN
 	1    3375 5400
@@
 F 0 "RV2" H 3680 1945 50  0000 R CNN
 F 1 "10K" H 3680 1855 50  0000 R CNN
-F 2 "Potentiometer_THT:Potentiometer_Piher_PT-6-V_Vertical" H 3750 1900 50  0001 C CNN
+F 2 "Potentiometer_THT:Potentiometer_Piher_PT-6-H_Horizontal" H 3750 1900 50  0001 C CNN
 F 3 "~" H 3750 1900 50  0001 C CNN
 	1    3750 1900

Commit message: Add eeprom load store capability
Parts:
- added J1: Microphone, openxcvr:jack3.5mm switched, symbol Connector:AudioJack2_Ground_Switch
- added J2: Mic, Connector_PinHeader_2.54mm:PinHeader_1x02_P2.54mm_Vertical, symbol Connector:Conn_01x02_Male
- added J3: Speaker, Connector_PinHeader_2.54mm:PinHeader_1x02_P2.54mm_Vertical, symbol Connector:Conn_01x02_Male
- added J4: Headphone, openxcvr:jack3.5mm switched, symbol Connector:AudioJack2_Ground_Switch
- added R2: 1K, Resistor_SMD:R_0805_2012Metric, symbol Device:R
- RV1: renamed from RV2; footprint Potentiometer_THT:Potentiometer_Piher_PT-6-H_Horizontal -> Potentiometer_THT:Potentiometer_Piher_PT-6-V_Vertical
- RV2: renamed from RV1; footprint Potentiometer_THT:Potentiometer_Piher_PT-6-H_Horizontal -> Potentiometer_THT:Potentiometer_Piher_PT-6-V_Vertical
- renumbered C9 to C10, C24 to C13, C13 to C14, C14 to C15, C15 to C16, C16 to C17, C17 to C18, C18 to C19, C10 to C9, R8 to R10, R9 to R11, R10 to R12, R2 to R3, R1 to R4, R3 to R5, R4 to R6, R5 to R7, R6 to R8, R7 to R9
Connections:
- net labels added: +5VA, PTT
- net labels removed: MIC_HDR, SPEAKER_HDR
- wire segments 86 -> 106
- no-connect marks 3 -> 5
Other:
- moved on the sheet: C13, C9, R3, R5, RV1

Commit message: update rev0.2 PCB
Parts:
- removed C16: 100u, Capacitor_Tantalum_SMD:CP_EIA-7343-31_Kemet-D, symbol Device:CP
- removed RV1, RV2: 10K, Potentiometer_THT:Potentiometer_Piher_PT-6-V_Vertical, symbol Device:R_POT_TRIM
- removed U2: LM386, Package_SO:SOIC-8_3.9x4.9mm_P1.27mm, symbol Amplifier_Audio:LM386
- added U2: TPA711, Package_SO:SOIC-8_3.9x4.9mm_P1.27mm, symbol xcvr_components:TPA711
- C15: value 47n -> 100n
- R9: value 10 -> 50k
Connections:
- wire segments 106 -> 112
- no-connect marks 5 -> 1
Other:
- moved on the sheet: C11, C12, C13, C14, C9, J3, J4, R10, R3, R5, R6, R7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

Commit message: Review and update schematic
Parts:
- added C50: 47p, Capacitor_SMD:C_0805_2012Metric, symbol Device:C
- R9: value 50k -> 47k
- U2: value TPA711 -> TPA711D
Connections:
- wire segments 112 -> 118
Changed lines of the file:
@@
 Connection ~ 3275 5675
 Connection ~ 3775 5050
-Connection ~ 4475 4950
+Connection ~ 3800 5450
+Connection ~ 4500 5450
+Connection ~ 4525 4950
 Connection ~ 4550 1650
 Connection ~ 4650 1550
@@
 Connection ~ 9450 4100
 Connection ~ 9450 5000
-NoConn ~ 1450 5350
+NoConn ~ 1550 4950
 Wire Wire Line
 	1350 5350 1350 5400
@@
 	3775 5450 3775 5050
 Wire Wire Line
+	3800 5450 3775 5450
+Wire Wire Line
+	3800 5800 3800 5450
+Wire Wire Line
 	3900 1650 4100 1650
 Wire Wire Line
-	3975 5450 3775 5450
-Wire Wire Line
-	4275 5450 4475 5450
+	3950 5800 3800 5800
+Wire Wire Line
+	3975 5450 3800 5450
+Wire Wire Line
+	4250 5800 4500 5800
+Wire Wire Line
+	4275 5450 4500 5450
 Wire Wire Line
 	4400 1650 4550 1650
 Wire Wire Line
-	4475 4950 4425 4950
-Wire Wire Line
-	4475 4950 4825 4950
-Wire Wire Line
-	4475 5450 4475 4950
+	4500 5450 4525 5450
+Wire Wire Line
+	4500 5800 4500 5450
+Wire Wire Line
+	4525 4950 4425 4950
+Wire Wire Line
+	4525 4950 4825 4950
+Wire Wire Line
+	4525 5450 4525 4950
 Wire Wire Line
 	4550 1650 4550 1950
@@
 P 5200 1950
 F 0 "R9" H 5270 1995 50  0000 L CNN
-F 1 "50k" H 5270 1905 50  0000 L CNN
+F 1 "47k" H 5270 1905 50  0000 L CNN
 F 2 "Resistor_SMD:R_0805_2012Metric" V 5130 1950 50  0001 C CNN
 F 3 "~" H 5200 1950 50  0001 C CNN
@@
 $EndComp
 $Comp
+L Device:C C50
+U 1 1 5F00647E
+P 4100 5800
+F 0 "C50" V 4351 5800 50  0000 C CNN
+F 1 "47p" V 4260 5800 50  0000 C CNN
+F 2 "Capacitor_SMD:C_0805_2012Metric" H 4138 5650 50  0001 C CNN
+F 3 "~" H 4100 5800 50  0001 C CNN
+	1    4100 5800
+	0    -1   -1   0
+$EndComp
+$Comp
 L Device:C C10
 U 1 1 5ED58F0A
@@
 P 5250 1250
 F 0 "U2" H 5250 1373 50  0000 C CNN
-F 1 "TPA711" H 5250 1282 50  0000 C CNN
+F 1 "TPA711D" H 5250 1282 50  0000 C CNN
 F 2 "Package_SO:SOIC-8_3.9x4.9mm_P1.27mm" H 4900 1250 50  0001 C CNN
 F 3 "https://www.ti.com/lit/ds/symlink/tpa711.pdf?ts=1590773198998" H 5250 1250 50  0001 C CNN

Commit message: Review schematic and PCB layout
Other:
- moved on the sheet: C12, C14, C50, R10, R6, R7, R8
Changed lines of the file:
@@
 $Descr A4 11693 8268
 encoding utf-8
-Sheet 3 7
+Sheet 5 7
 Title "Open XCVR"
-Date "2020-01-26"
-Rev "0.1"
+Date "2020-06-14"
+Rev "0.2"
 Comp "Jon Dawson"
 Comment1 ""
@@
 Connection ~ 2450 5050
 Connection ~ 3150 1650
-Connection ~ 3275 4275
-Connection ~ 3275 4725
-Connection ~ 3275 4850
-Connection ~ 3275 5225
-Connection ~ 3275 5675
-Connection ~ 3775 5050
+Connection ~ 3250 4050
+Connection ~ 3250 4550
+Connection ~ 3250 4700
+Connection ~ 3250 5250
+Connection ~ 3250 5650
+Connection ~ 3800 5050
 Connection ~ 3800 5450
-Connection ~ 4500 5450
-Connection ~ 4525 4950
 Connection ~ 4550 1650
+Connection ~ 4600 4950
+Connection ~ 4600 5450
 Connection ~ 4650 1550
 Connection ~ 5800 1650
@@
 	2450 4700 2450 5050
 Wire Wire Line
-	2450 5050 2875 5050
+	2450 5050 2850 5050
 Wire Wire Line
 	2850 1650 3150 1650
 Wire Wire Line
-	2850 5225 3275 5225
-Wire Wire Line
-	2850 5300 2850 5225
-Wire Wire Line
-	2850 5600 2850 5675
-Wire Wire Line
-	2850 5675 3275 5675
-Wire Wire Line
-	2875 4275 2875 4350
-Wire Wire Line
-	2875 4275 3275 4275
-Wire Wire Line
-	2875 4650 2875 4725
-Wire Wire Line
-	2875 4725 3275 4725
+	2850 4050 3250 4050
+Wire Wire Line
+	2850 4150 2850 4050
+Wire Wire Line
+	2850 4450 2850 4550
+Wire Wire Line
+	2850 4550 3250 4550
+Wire Wire Line
+	2850 5250 3250 5250
+Wire Wire Line
+	2850 5300 2850 5250
+Wire Wire Line
+	2850 5600 2850 5650
+Wire Wire Line
+	2850 5650 3250 5650
 Wire Wire Line
 	3150 1650 3150 1750
@@
 	3150 2050 3150 2100
 Wire Wire Line
-	3175 5050 3375 5050
-Wire Wire Line
-	3275 4200 3275 4275
-Wire Wire Line
-	3275 4275 3275 4350
-Wire Wire Line
-	3275 4650 3275 4725
-Wire Wire Line
-	3275 4725 3275 4850
-Wire Wire Line
-	3275 4850 3275 5225
-Wire Wire Line
-	3275 4850 3825 4850
-Wire Wire Line
-	3275 5225 3275 5300
-Wire Wire Line
-	3275 5600 3275 5675
-Wire Wire Line
-	3275 5675 3275 5750
-Wire Wire Line
-	3675 5050 3775 5050
-Wire Wire Line
-	3775 5050 3825 5050
-Wire Wire Line
-	3775 5450 3775 5050
-Wire Wire Line
-	3800 5450 3775 5450
+	3150 5050 3400 5050
+Wire Wire Line
+	3250 4000 3250 4050
+Wire Wire Line
+	3250 4050 3250 4150
+Wire Wire Line
+	3250 4450 3250 4550
+Wire Wire Line
+	3250 4550 3250 4700
+Wire Wire Line
+	3250 4700 3250 5250
+Wire Wire Line
+	3250 4700 3800 4700
+Wire Wire Line
+	3250 5250 3250 5300
+Wire Wire Line
+	3250 5600 3250 5650
+Wire Wire Line
+	3250 5650 3250 5750
+Wire Wire Line
+	3700 5050 3800 5050
+Wire Wire Line
+	3800 4850 3800 4700
+Wire Wire Line
+	3800 5050 3900 5050
+Wire Wire Line
+	3800 5450 3800 5050
 Wire Wire Line
 	3800 5800 3800 5450
@@
 	3900 1650 4100 1650
 Wire Wire Line
-	3950 5800 3800 5800
-Wire Wire Line
-	3975 5450 3800 5450
-Wire Wire Line
-	4250 5800 4500 5800
-Wire Wire Line
-	4275 5450 4500 5450
+	3900 4850 3800 4850
+Wire Wire Line
+	4000 5450 3800 5450
+Wire Wire Line
+	4000 5800 3800 5800
+Wire Wire Line
+	4300 5450 4600 5450
+Wire Wire Line
+	4300 5800 4600 5800
 Wire Wire Line
 	4400 1650 4550 1650
 Wire Wire Line
-	4500 5450 4525 5450
-Wire Wire Line
-	4500 5800 4500 5450
-Wire Wire Line
-	4525 4950 4425 4950
-Wire Wire Line
-	4525 4950 4825 4950
-Wire Wire Line
-	4525 5450 4525 4950
+	4500 4950 4600 4950
 Wire Wire Line
 	4550 1650 4550 1950
@@
 Wire Wire Line
 	4600 2450 4600 2600
+Wire Wire Line
+	4600 4950 4900 4950
+Wire Wire Line
+	4600 5450 4600 4950
+Wire Wire Line
+	4600 5800 4600 5450
 Wire Wire Line
 	4650 1350 4650 1550
@@
 Text GLabel 2150 4850 2    50   Output ~ 0
 PTT
-Text GLabel 4825 4950 2    50   Output ~ 0
+Text GLabel 4900 4950 2    50   Output ~ 0
 MIC
 $Comp
@@
 L power:+3V3 #PWR028
 U 1 1 5E3553EF
-P 3275 4200
-F 0 "#PWR028" H 3275 4050 50  0001 C CNN
-F 1 "+3V3" H 3290 4373 50  0000 C CNN
-F 2 "" H 3275 4200 50  0001 C CNN
-F 3 "" H 3275 4200 50  0001 C CNN
-	1    3275 4200
+P 3250 4000
+F 0 "#PWR028" H 3250 3850 50  0001 C CNN
+F 1 "+3V3" H 3265 4173 50  0000 C CNN
+F 2 "" H 3250 4000 50  0001 C CNN
+F 3 "" H 3250 4000 50  0001 C CNN
+	1    3250 4000
 	1    0    0    -1
 $EndComp
@@
 L power:GND #PWR029
 U 1 1 5E3549BE
-P 3275 5750
-F 0 "#PWR029" H 3275 5500 50  0001 C CNN
-F 1 "GND" H 3280 5577 50  0000 C CNN
-F 2 "" H 3275 5750 50  0001 C CNN
-F 3 "" H 3275 5750 50  0001 C CNN
-	1    3275 5750
+P 3250 5750
+F 0 "#PWR029" H 3250 5500 50  0001 C CNN
+F 1 "GND" H 3255 5577 50  0000 C CNN
+F 2 "" H 3250 5750 50  0001 C CNN
+F 3 "" H 3250 5750 50  0001 C CNN
+	1    3250 5750
 	1    0    0    -1
 $EndComp
@@
 L Device:R R6
 U 1 1 5E2E0080
-P 3275 4500
-F 0 "R6" H 3345 4545 50  0000 L CNN
-F 1 "100K" H 3345 4455 50  0000 L CNN
-F 2 "Resistor_SMD:R_0805_2012Metric" V 3205 4500 50  0001 C CNN
-F 3 "~" H 3275 4500 50  0001 C CNN
-	1    3275 4500
+P 3250 4300
+F 0 "R6" H 3320 4345 50  0000 L CNN
+F 1 "100K" H 3320 4255 50  0000 L CNN
+F 2 "Resistor_SMD:R_0805_2012Metric" V 3180 4300 50  0001 C CNN
+F 3 "~" H 3250 4300 50  0001 C CNN
+	1    3250 4300
 	1    0    0    -1
 $EndComp
@@
 L Device:R R7
 U 1 1 5E2E5F41
-P 3275 5450
-F 0 "R7" H 3345 5495 50  0000 L CNN
-F 1 "100K" H 3345 5405 50  0000 L CNN
-F 2 "Resistor_SMD:R_0805_2012Metric" V 3205 5450 50  0001 C CNN
-F 3 "~" H 3275 5450 50  0001 C CNN
-	1    3275 5450
+P 3250 5450
+F 0 "R7" H 3320 5495 50  0000 L CNN
+F 1 "100K" H 3320 5405 50  0000 L CNN
+F 2 "Resistor_SMD:R_0805_2012Metric" V 3180 5450 50  0001 C CNN
+F 3 "~" H 3250 5450 50  0001 C CNN
+	1    3250 5450
 	1    0    0    -1
 $EndComp
@@
 L Device:R R8
 U 1 1 5E2E0764
-P 3525 5050
-F 0 "R8" V 3731 5050 50  0000 C CNN
-F 1 "1K" V 3640 5050 50  0000 C CNN
-F 2 "Resistor_SMD:R_0805_2012Metric" V 3455 5050 50  0001 C CNN
-F 3 "~" H 3525 5050 50  0001 C CNN
-	1    3525 5050
+P 3550 5050
+F 0 "R8" V 3756 5050 50  0000 C CNN
+F 1 "1K" V 3665 5050 50  0000 C CNN
+F 2 "Resistor_SMD:R_0805_2012Metric" V 3480 5050 50  0001 C CNN
+F 3 "~" H 3550 5050 50  0001 C CNN
+	1    3550 5050
 	0    -1   -1   0
 $EndComp
@@
 L Device:R R10
 U 1 1 5E2E16E9
-P 4125 5450
-F 0 "R10" V 4331 5450 50  0000 C CNN
-F 1 "1M" V 4240 5450 50  0000 C CNN
-F 2 "Resistor_SMD:R_0805_2012Metric" V 4055 5450 50  0001 C CNN
-F 3 "~" H 4125 5450 50  0001 C CNN
-	1    4125 5450
+P 4150 5450
+F 0 "R10" V 4356 5450 50  0000 C CNN
+F 1 "1M" V 4265 5450 50  0000 C CNN
+F 2 "Resistor_SMD:R_0805_2012Metric" V 4080 5450 50  0001 C CNN
+F 3 "~" H 4150 5450 50  0001 C CNN
+	1    4150 5450
 	0    -1   -1   0
 $EndComp
@@
 U 1 1 5ED3BE3F
 P 5200 1950
-F 0 "R9" H 5270 1995 50  0000 L CNN
-F 1 "47k" H 5270 1905 50  0000 L CNN
+F 0 "R9" V 5000 1900 50  0000 L CNN
+F 1 "47k" V 5100 1850 50  0000 L CNN
 F 2 "Resistor_SMD:R_0805_2012Metric" V 5130 1950 50  0001 C CNN
 F 3 "~" H 5200 1950 50  0001 C CNN
@@
 $EndComp
 $Comp
+L Device:C C12
+U 1 1 5E2F8697
+P 2850 4300
+F 0 "C12" H 2965 4345 50  0000 L CNN
+F 1 "100n" H 2965 4255 50  0000 L CNN
+F 2 "Capacitor_SMD:C_0805_2012Metric" H 2888 4150 50  0001 C CNN
+F 3 "~" H 2850 4300 50  0001 C CNN
+	1    2850 4300
+	1    0    0    -1
+$EndComp
+$Comp
 L Device:C C11
 U 1 1 5E2F9F9C
@@
 $EndComp
 $Comp
-L Device:C C12
-U 1 1 5E2F8697
-P 2875 4500
-F 0 "C12" H 2990 4545 50  0000 L CNN
-F 1 "100n" H 2990 4455 50  0000 L CNN
-F 2 "Capacitor_SMD:C_0805_2012Metric" H 2913 4350 50  0001 C CNN
-F 3 "~" H 2875 4500 50  0001 C CNN
-	1    2875 4500
-	1    0    0    -1
-$EndComp
-$Comp
 L Device:C C14
 U 1 1 5E2FC763
-P 3025 5050
-F 0 "C14" V 3276 5050 50  0000 C CNN
-F 1 "100n" V 3185 5050 50  0000 C CNN
-F 2 "Capacitor_SMD:C_0805_2012Metric" H 3063 4900 50  0001 C CNN
-F 3 "~" H 3025 5050 50  0001 C CNN
-	1    3025 5050
+P 3000 5050
+F 0 "C14" V 3251 5050 50  0000 C CNN
+F 1 "100n" V 3160 5050 50  0000 C CNN
+F 2 "Capacitor_SMD:C_0805_2012Metric" H 3038 4900 50  0001 C CNN
+F 3 "~" H 3000 5050 50  0001 C CNN
+	1    3000 5050
 	0    -1   -1   0
 $EndComp
@@
 L Device:C C50
 U 1 1 5F00647E
-P 4100 5800
-F 0 "C50" V 4351 5800 50  0000 C CNN
-F 1 "47p" V 4260 5800 50  0000 C CNN
-F 2 "Capacitor_SMD:C_0805_2012Metric" H 4138 5650 50  0001 C CNN
-F 3 "~" H 4100 5800 50  0001 C CNN
-	1    4100 5800
+P 4150 5800
+F 0 "C50" V 4401 5800 50  0000 C CNN
+F 1 "47p" V 4310 5800 50  0000 C CNN
+F 2 "Capacitor_SMD:C_0805_2012Metric" H 4188 5650 50  0001 C CNN
+F 3 "~" H 4150 5800 50  0001 C CNN
+	1    4150 5800
 	0    -1   -1   0
 $EndComp
@@
 L Amplifier_Operational:MCP6002-xSN U3
 U 1 1 5E2DD833
-P 4125 4950
-F 0 "U3" H 4125 5316 50  0000 C CNN
-F 1 "MCP6002-xSN" H 4125 5225 50  0000 C CNN
-F 2 "Package_SO:SOIC-8_3.9x4.9mm_P1.27mm" H 4125 4950 50  0001 C CNN
-F 3 "http://ww1.microchip.com/downloads/en/DeviceDoc/21733j.pdf" H 4125 4950 50  0001 C CNN
-	1    4125 4950
-	1    0    0    -1
-$EndComp
+P 4200 4950
+F 0 "U3" H 4200 5316 50  0000 C CNN
+F 1 "MCP6002-xSN" H 4200 5225 50  0000 C CNN
+F 2 "Package_SO:SOIC-8_3.9x4.9mm_P1.27mm" H 4200 4950 50  0001 C CNN
+F 3 "http://ww1.microchip.com/downloads/en/DeviceDoc/21733j.pdf" H 4200 4950 50  0001 C CNN
+	1    4200 4950
+	1    0    0    -1
+$EndComp

Commit message: PCB reviewed and updated
Parts:
- added C52: 100n, Capacitor_SMD:C_0805_2012Metric, symbol Device:C
- added C53: 100u, Capacitor_Tantalum_SMD:CP_EIA-7343-31_Kemet-D, symbol Device:CP
- added R45, R46: 100K, Resistor_SMD:R_0805_2012Metric, symbol Device:R
- added R47: 1K, Resistor_SMD:R_0805_2012Metric, symbol Device:R
Connections:
- wire segments 118 -> 141
Other:
- moved on the sheet: C10, C13, C9, J3, J4, R3, R5
